File: GrowChamberPCB/GrowChamberPCB.kicad_sch (KiCad schematic)
At the start: 28 parts, among them J1 Screw_Terminal_01x02, J2 Conn_01x03_Pin, J4 Conn_01x02_Socket, U2 MCP1826S, U4 TC4428xOA, U5 W25Q128JVS

Commit message: bunch o stuff
Parts:
- added C12, C17: 0.1uF, symbol Device:C
- added C13: 22uF, symbol Device:C
- added C14: 1uF, symbol Device:C
- added C15, C16: DNP, symbol Device:C
- added C20: 100nF, symbol Device:C
- added J3: TYPE-C-31-M-12, Connector_USB:USB_C_Receptacle_HRO_TYPE-C-31-M-12, symbol Custom_Library:TYPE-C-31-M-12
- added JP1: SD Card Detect, symbol Jumper:Jumper_2_Small_Open
- added R10, R9: 5.1K, symbol Device:R
- added R11, R6: 10k, symbol Device:R
- added R12, R13: 10K, symbol Device:R
- added R7, R8: 22, symbol Device:R
- added SW1: BootMode, symbol Switch:SW_Push
- added SW2: Reset, symbol Switch:SW_Push
- added U1: ESP32-S3-WROOM-1U, ESP32-S3-WROOM-1U:XCVR_ESP32-S3-WROOM-1U, symbol Custom_Library:ESP32-S3-WROOM-1U
- added U3: USBLC6-2SC6, Package_TO_SOT_SMD:SOT-23-6, symbol Power_Protection:USBLC6-2SC6
- added U6: CR2013-MI2120, Display:CR2013-MI2120, symbol Driver_Display:CR2013-MI2120
- J2: value Conn_01x03_Pin -> UART Upload
- J4: value Conn_01x02_Socket -> Piezo Connector
Connections:
- net 3.3V: now also U5.8 (VCC), C12.2, C13.2, C20.2, R11.1, R12.1, R13.2, R6.2, U1.2 (3V3), U6.1 (VCC), U6.8 (LED)
- net GPIO11: now reaches U4.2 (IN_A)
- net GPIO11: now also U4.4 (IN_B), U1.19 (IO11)
- net MISO: now reaches U5.2 (DO/IO_{1})
- net MISO: now also U1.35 (IO42), U6.12 (SD_MISO), U6.9 (MISO)
- net at U5.3 (~{WP}/IO_{2}): now also U5.7 (~{HOLD}/~{RESET}/IO_{3}), R13.1
- net MOSI: now reaches U5.5 (DI/IO_{0})
- net MOSI: now also U1.34 (IO41), U6.11 (SD_MOSI), U6.6 (MOSI)
- net SCK: now reaches U5.6 (CLK)
- net SCK: now also U1.33 (IO40), U6.13 (SD_SCK), U6.7 (SCK)
- net CS_Memory / GPIO4 renamed CS_Memory
- net CS_Memory: now also U1.25 (IO48)
- net ESP32-S3-Wroom-1U/RXD0 renamed RXD0
- net RXD0: now also U1.36 (RXD0)
- net ESP32-S3-Wroom-1U/TXD0 renamed TXD0
- net TXD0: now also U1.37 (TXD0)
- net Gnd renamed GND
- net GND: now also C12.1, C13.1, C14.1, C15.2, C16.2, C17.1, C20.1, J3.A1_B12 (GND), J3.B1_A12 (GND), J3.S1 (SHIELD), J3.S2 (SHIELD), J3.S3 (SHIELD), J3.S4 (SHIELD), R10.2, R9.1, SW1.2, SW2.2, U1.1 (GND), U1.40 (GND), U1.41_1 (GND), U1.41_2 (GND), U1.41_3 (GND), U1.41_4 (GND), U1.41_5 (GND), U1.41_6 (GND), U1.41_7 (GND), U1.41_8 (GND), U1.41_9 (GND), U3.2 (GND), U6.2 (GND)
- new net: R7.1, U1.13 (IO19)
- new net: R8.1, U1.14 (IO20)
- new net: R11.2, SW1.1, U1.27 (IO0)
- new net: C14.2, C17.2, R6.1, SW2.1, U1.3 (EN)
- new net: JP1.2 (B), R12.2, U6.14 (FLASH_CD)
- new net: C15.1, R8.2, U3.1 (I/O1)
- new net: J3.A5 (CC1), R9.2
- new net: J3.B5 (CC2), R10.1
- new net: C16.1, R7.2, U3.3 (I/O2)
- new net CS_Display: U1.31 (IO38), U6.3 (~{CS})
- new net CS_SD: U1.23 (IO21), U6.10 (SD_CS)
- new net D+: J3.A7 (DN1), J3.B7 (DN2), U3.6 (I/O1)
- new net D-: J3.A6 (DP1), J3.B6 (DP2), U3.4 (I/O2)
- new net DC_Display: U1.32 (IO39), U6.5 (D/~{C})
- new net Display_Reset: U1.24 (IO47), U6.4 (RESET)
- new net GPIO10: U1.18 (IO10)
- new net GPIO12: U1.20 (IO12)
- new net GPIO13: U1.21 (IO13)
- new net GPIO14: U1.22 (IO14)
- new net GPIO15: U1.8 (IO15)
- new net GPIO16: U1.9 (IO16)
- new net GPIO17: U1.10 (IO17)
- new net GPIO18: U1.11 (IO18)
- new net GPIO35: U1.28 (IO35)
- new net GPIO36: U1.29 (IO36)
- new net GPIO37: U1.30 (IO37)
- new net GPIO4: U1.4 (IO4)
- new net GPIO45: U1.26 (IO45)
- new net GPIO46: U1.16 (IO46)
- new net GPIO5: U1.5 (IO5)
- new net GPIO6: U1.6 (IO6)
- new net GPIO7: U1.7 (IO7)
- new net GPIO8: U1.12 (IO8)
- new net GPIO9: U1.17 (IO9)
- new net SD_Detect: JP1.1 (A), U1.15 (IO3)
- new net VBUS: J3.A4_B9 (VBUS), J3.B4_A9 (VBUS), U3.5 (VBUS)
- no-connect marks 0 -> 2
Other:
- removed sheet ESP32-S3-Wroom-1U
- removed sheet USB Connector
- added sheet MOSFET_Switching (MOSFET_Switching.kicad_sch)
- note added: "Display"
- note added: "Extra Memory"
- note added: "GPIO46 - Don't pull high through a peripheral."
- note added: "Piezoelectric Mister"
- note added: "USB Port"
- moved on the sheet: C18, C19, J2, J4, JP2, JP3, U4, U5

Commit message: Lots of things, MOSFET switch schematic confirmed
Parts:
- removed J2: UART Upload, symbol Connector:Conn_01x03_Pin
- removed J4: Piezo Connector, symbol Connector:Conn_01x02_Socket
- added D2, D3, D4, D5, D6, D7: 1N4007, Diode_SMD:D_SMA, symbol Diode:1N4007
- added J6: Screw_Terminal_01x20, symbol Connector:Screw_Terminal_01x20
- added Q2, Q3, Q4, Q5, Q6, Q7: IRLML6244, Package_TO_SOT_SMD:SOT-23, symbol Transistor_FET:IRLML6244
- added R16, R18, R20, R22, R24, R26: 100, symbol Device:R
- added R17, R19, R21, R23, R25, R27: 10K, symbol Device:R
Connections:
- net 12V: now also D2.2 (A), D3.2 (A), D4.2 (A), D5.2 (A), D6.2 (A), D7.2 (A), J6.18 (Pin_18)
- net 5V: now also J6.19 (Pin_19)
- net GND: now also J6.20 (Pin_20), Q2.2 (S), Q3.2 (S), Q4.2 (S), Q5.2 (S), Q6.2 (S), Q7.2 (S), R17.1, R19.1, R21.1, R23.1, R25.1, R27.1
- net GPIO13: now also R16.2
- net GPIO14: now also R18.2
- net GPIO15: now also R20.2
- net GPIO16: now also R22.2
- net GPIO17: now also R24.2
- net GPIO18: now also R26.2
- net GPIO4: now also J6.7 (Pin_7)
- net RXD0: now also J6.1 (Pin_1)
- net TXD0: now also J6.2 (Pin_2)
- net GPIO2: now reaches U1.38 (IO2)
- net GPIO2: now also J6.8 (Pin_8)
- net GPIO1: now reaches U1.39 (IO1)
- net GPIO1: now also J6.9 (Pin_9)
- net Piezo2: now reaches U4.5 (OUT_B)
- net Piezo2: now also J6.10 (Pin_10)
- net Piezo1: now reaches U4.7 (~{OUT_A})
- net Piezo1: now also J6.11 (Pin_11)
- new net: Q3.1 (G), R18.1, R19.2
- new net: Q5.1 (G), R22.1, R23.2
- new net: Q7.1 (G), R26.1, R27.2
- new net: Q2.1 (G), R16.1, R17.2
- new net: Q6.1 (G), R24.1, R25.2
- new net: Q4.1 (G), R20.1, R21.2
- new net DrainSol: D4.1 (K), J6.14 (Pin_14), Q4.3 (D)
- new net FoggerSol: D5.1 (K), J6.15 (Pin_15), Q5.3 (D)
- new net GlycolSol: D2.1 (K), J6.12 (Pin_12), Q2.3 (D)
- new net LEDs: D7.1 (K), J6.17 (Pin_17), Q7.3 (D)
- new net RadiatorFans: D6.1 (K), J6.16 (Pin_16), Q6.3 (D)
- new net WaterSol: D3.1 (K), J6.13 (Pin_13), Q3.3 (D)
Other:
- removed sheet MOSFET_Switching
- added sheet Heater Switching (Heater Switching.kicad_sch)
- note added: "1, 2, 4 for Soil Moisture Sensors"
- moved on the sheet: C1, C10, C11, C18, C19, C2, C20, C3, C4, C5, C6, C7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

Commit message: Working on faceplate
Parts:
- removed J6: Screw_Terminal_01x20, symbol Connector:Screw_Terminal_01x20
- added J11: Conn_01x24_Pin, symbol Connector:Conn_01x24_Pin
- added J4: Optocoupler to GPIO, symbol Connector:Screw_Terminal_01x02
- added J8: To Relay Board, symbol Connector:Screw_Terminal_01x02
- added Q1: IRLML6244, Package_TO_SOT_SMD:SOT-23, symbol Transistor_FET:IRLML6244
- added R14: 10K, symbol Device:R
- added R15: 100, symbol Device:R
- U6: footprint Display:CR2013-MI2120 -> Connector_PinHeader_2.54mm:PinHeader_2x07_P2.54mm_Vertical
Connections:
- net 12V: now also J11.21 (Pin_21), J8.1 (Pin_1)
- net 3.3V: now also J11.19 (Pin_19)
- net 5V: now also J11.20 (Pin_20)
- net DrainSol: now also J11.8 (Pin_8)
- net FoggerSol: now also J11.7 (Pin_7)
- net GND: now also J11.18 (Pin_18), J4.1 (Pin_1), Q1.2 (S), R14.1
- net GPIO1: now also J11.13 (Pin_13)
- net GPIO2: now also J11.14 (Pin_14)
- net GPIO4: now also J11.15 (Pin_15)
- net GlycolSol: now also J11.10 (Pin_10)
- net Piezo1: now also J11.11 (Pin_11)
- net Piezo2: now also J11.12 (Pin_12)
- net RXD0: now also J11.23 (Pin_23)
- net RadiatorFans: now also J11.6 (Pin_6)
- net TXD0: now also J11.22 (Pin_22)
- net WaterSol: now also J11.9 (Pin_9)
- net GPIO10 renamed External_Fan_PWM
- net External_Fan_PWM: now also J11.4 (Pin_4)
- net GPIO11 renamed Fogger_PWM
- net GPIO12 renamed Heater_Switch
- net Heater_Switch: now also R15.2
- net GPIO35: no longer names the net of U1.28 (IO35)
- net GPIO36: no longer names the net of U1.29 (IO36)
- net GPIO37: no longer names the net of U1.30 (IO37)
- net GPIO5 renamed SDA
- net SDA: now also J11.17 (Pin_17)
- net GPIO6 renamed SCL
- net SCL: now also J11.16 (Pin_16)
- net GPIO7 renamed Drain_Level
- net Drain_Level: now also J11.5 (Pin_5)
- net GPIO8 renamed Fogger_Basin_Float_Switch
- net Fogger_Basin_Float_Switch: now also J11.24 (Pin_24)
- net GPIO9 renamed KSD_Fault
- net KSD_Fault: now also J4.2 (Pin_2)
- new net: Q1.1 (G), R14.2, R15.1
- new net: J8.2 (Pin_2), Q1.3 (D)
- no-connect marks 2 -> 5
Other:
- sheet Heater Switching renamed Heater Switching Board
- added sheet Faceplate_Board (Faceplate_Board.kicad_sch)
- sheet Heater Switching Board ports: added none; removed GPIO
- note added: "2 - MOSFET Drain 1 - 12V"
- note added: "LEDs on separate connector"
- moved on the sheet: R11, SW1
