File: GrowChamberPCB/GrowChamberPCB.kicad_sch (KiCad schematic)
At the start: 78 parts, among them J1 Screw_Terminal_01x02, J11 Conn_01x24_Pin, J3 TYPE-C-31-M-12, J4 Optocoupler to GPIO, J8 To Relay Board, Q1 IRLML6244, Q2 IRLML6244, Q3 IRLML6244, Q4 IRLML6244, Q5 IRLML6244, Q6 IRLML6244, Q7 IRLML6244, SW1 BootMode, SW2 Reset, U1 ESP32-S3-WROOM-1U, U2 MCP1826S, U3 USBLC6-2SC6, U4 TC4428xOA, U5 W25Q128JVS, U6 CR2013-MI2120

Commit message: Working on faceplate
Parts:
- removed J4: Optocoupler to GPIO, symbol Connector:Screw_Terminal_01x02
- removed J8: To Relay Board, symbol Connector:Screw_Terminal_01x02
- removed SW1: BootMode, symbol Switch:SW_Push
- added J7: Screw_Terminal_01x05, symbol Connector:Screw_Terminal_01x05
- added SW5: BootSwitch, symbol Switch:SW_Push
Connections:
- net GPIO45 is gone; now on net Fan_Tach: U1.26 (IO45)
- net 12V: now also J7.4 (Pin_4)
- net 5V: now also J7.3 (Pin_3)
- net GND: now also J7.2 (Pin_2), SW5.2
- net KSD_Fault: now also J7.1 (Pin_1)
- net BootMode: now reaches R11.2, U1.27 (IO0)
- net BootMode: now also J11.1 (Pin_1), SW5.1
- net Reset_SW: now reaches C14.2, C17.2, R6.1, SW2.1, U1.3 (EN)
- net Reset_SW: now also J11.2 (Pin_2)
- net at Q1.3 (D): now also J7.5 (Pin_5)
- net Fan_Tach: now reaches J11.3 (Pin_3)
Other:
- moved on the sheet: J11, SW2

Commit message: final schematic
Parts:
- added D8: 1N4007, Diode_SMD:D_SMA, symbol Diode:1N4007
- added J8: Screw_Terminal_01x02, symbol Connector:Screw_Terminal_01x02
- added Q8: IRLML6244, Package_TO_SOT_SMD:SOT-23, symbol Transistor_FET:IRLML6244
- added R30: 100, symbol Device:R
- added R31: 10K, symbol Device:R
- Q7: value IRLML6244 -> IRLR8721; footprint Package_TO_SOT_SMD:SOT-23 -> Package_TO_SOT_SMD:TO-252-2
- U1: footprint ESP32-S3-WROOM-1U:XCVR_ESP32-S3-WROOM-1U -> (none)
Connections:
- net 12V: now also D2.1 (K), D3.1 (K), D4.1 (K), D5.1 (K), D6.1 (K), D7.1 (K), D8.1 (K); no longer D2.2 (A), D3.2 (A), D4.2 (A), D5.2 (A), D6.2 (A), D7.2 (A)
- net 3.3V: no longer J11.19 (Pin_19)
- net DrainSol: now also D4.2 (A); no longer D4.1 (K)
- net FoggerSol: now also D5.2 (A); no longer D5.1 (K)
- net GND: now also J8.2 (Pin_2), Q8.2 (S), R31.1
- net GPIO46: now also R30.2
- net GlycolSol: now also D2.2 (A); no longer D2.1 (K)
- net LEDs: now also D7.2 (A), J8.1 (Pin_1); no longer D7.1 (K)
- net RadiatorFans: now also D6.2 (A); no longer D6.1 (K)
- net WaterSol: now also D3.2 (A); no longer D3.1 (K)
- new net: Q8.1 (G), R30.1, R31.2
- new net Circ_Fan: D8.2 (A), J11.19 (Pin_19), Q8.3 (D)
Other:
- moved on the sheet: D2, D3, D4, D5, D6, D7

Commit message: Assigning footprints and stuff
Parts:
- removed J11: Conn_01x24_Pin, symbol Connector:Conn_01x24_Pin
- added J27: Conn_01x26_Pin, symbol Connector:Conn_01x26_Pin
- added R32, R33: 10k, symbol Device:R
- C1: footprint (none) -> Capacitor_SMD:C_0805_2012Metric; MFG Part Number (none) -> GRM21BR61E226ME44L; Type (SMD/thru-hole, etc.) (none) -> SMD
- C4: footprint (none) -> Capacitor_SMD:C_0603_1608Metric; MFG Part Number (none) -> GRM188R71C105KA12D
- J3: Package Package -> (none); Package/Footprint (none) -> Package
- L1: value 3.9 or 3.3 -> 3.9
- U1: Package SMD-41 Espressif Systems -> (none); Package/Footprint (none) -> SMD-41 Espressif Systems
Connections:
- net 12V: now also J27.23 (Pin_23)
- net 3.3V: now also R32.1, R33.1
- net 5V: now also J27.22 (Pin_22)
- net BootMode: now also J27.3 (Pin_3)
- net Circ_Fan: now also J27.21 (Pin_21)
- net DrainSol: now also J27.10 (Pin_10)
- net Drain_Level: now also J27.7 (Pin_7)
- net External_Fan_PWM: now also J27.6 (Pin_6)
- net Fan_Tach: now also J27.5 (Pin_5)
- net FoggerSol: now also J27.9 (Pin_9)
- net Fogger_Basin_Float_Switch: now also J27.26 (Pin_26)
- net GPIO1: now also J27.15 (Pin_15)
- net GPIO2: now also J27.16 (Pin_16)
- net GPIO4: now also J27.17 (Pin_17)
- net GlycolSol: now also J27.12 (Pin_12), J27.20 (Pin_20)
- net Piezo1: now also J27.13 (Pin_13)
- net Piezo2: now also J27.14 (Pin_14)
- net RXD0: now also J27.25 (Pin_25)
- net Reset_SW: now also J27.4 (Pin_4)
- net SCL: now also J27.18 (Pin_18), R33.2
- net SDA: now also J27.19 (Pin_19), R32.2
- net TXD0: now also J27.24 (Pin_24)
- net WaterSol: now also J27.11 (Pin_11)
- net RadiatorFans renamed Heater Fans
- net Heater Fans: now also J27.8 (Pin_8)
Other:
- note added: "Place capacitors within 1mm of IN/GND pins."
- note removed: "Make sure C1 and C4 have an RMS current rating above 1.5A"

Commit message: struggling to make BOM
Parts:
- removed J8: Screw_Terminal_01x02, symbol Connector:Screw_Terminal_01x02
- removed JP1: SD Card Detect, symbol Jumper:Jumper_2_Small_Open
- removed Q8: IRLML6244, Package_TO_SOT_SMD:SOT-23, symbol Transistor_FET:IRLML6244
- removed R12: 10K, symbol Device:R
- added J10: Screw_Terminal_01x03, symbol Connector:Screw_Terminal_01x03
- added Q9: IRLML6244, symbol Transistor_FET:IRLML6244
- C1: footprint Capacitor_SMD:C_0805_2012Metric -> (none)
- C4: footprint Capacitor_SMD:C_0603_1608Metric -> (none)
- D2, D3, D4, D5, D6, D7, D8: footprint Diode_SMD:D_SMA -> (none)
- MP2393GTL-Z1: footprint Package_TO_SOT_SMD:SOT-583-8 -> (none)
- Q1, Q2, Q3, Q4, Q5, Q6: footprint Package_TO_SOT_SMD:SOT-23 -> (none)
- Q7: footprint Package_TO_SOT_SMD:TO-252-2 -> (none)
- U2: footprint Package_TO_SOT_SMD:SOT-223-3_TabPin2 -> (none)
- U3: footprint Package_TO_SOT_SMD:SOT-23-6 -> (none)
- U4: footprint Package_SO:SOIC-8_3.9x4.9mm_P1.27mm -> (none)
- U5: footprint Package_SO:SOIC-8_5.3x5.3mm_P1.27mm -> (none)
- U6: footprint Connector_PinHeader_2.54mm:PinHeader_2x07_P2.54mm_Vertical -> (none)
Connections:
- net 12V: now also J10.3 (Pin_3); no longer J27.23 (Pin_23)
- net 5V: now also J27.23 (Pin_23); no longer J27.22 (Pin_22)
- net BootMode: now also J27.5 (Pin_5); no longer J27.3 (Pin_3)
- net Circ_Fan: now also J27.22 (Pin_22), Q1.3 (D); no longer J27.21 (Pin_21)
- net DrainSol: now also J27.12 (Pin_12); no longer J27.10 (Pin_10)
- net Drain_Level: now also J27.9 (Pin_9); no longer J27.7 (Pin_7)
- net External_Fan_PWM: now also J27.8 (Pin_8); no longer J27.6 (Pin_6)
- net Fan_Tach: now also J27.7 (Pin_7); no longer J27.5 (Pin_5)
- net FoggerSol: now also J27.11 (Pin_11); no longer J27.9 (Pin_9)
- net GND: now also J10.2 (Pin_2), Q9.2 (S)
- net GPIO1: now also J27.17 (Pin_17); no longer J27.15 (Pin_15)
- net GPIO2: now also J27.18 (Pin_18); no longer J27.16 (Pin_16)
- net GPIO4: now also J27.19 (Pin_19); no longer J27.17 (Pin_17)
- net GlycolSol: now also J27.14 (Pin_14); no longer J27.12 (Pin_12), J27.20 (Pin_20)
- net Heater Fans: now also J27.10 (Pin_10); no longer J27.8 (Pin_8)
- net LEDs: now also J10.1 (Pin_1)
- net Piezo1: now also J27.15 (Pin_15); no longer J27.13 (Pin_13)
- net Piezo2: now also J27.16 (Pin_16); no longer J27.14 (Pin_14)
- net Reset_SW: now also J27.6 (Pin_6); no longer J27.4 (Pin_4)
- net SCL: now also J27.20 (Pin_20); no longer J27.18 (Pin_18)
- net SDA: now also J27.21 (Pin_21); no longer J27.19 (Pin_19)
- net WaterSol: now also J27.13 (Pin_13); no longer J27.11 (Pin_11)
- net at R30.1, R31.2: now also Q1.1 (G)
- net at R14.2, R15.1: now also Q9.1 (G); no longer Q1.1 (G)
- net Heater_On: now reaches J7.5 (Pin_5)
- net Heater_On: now also J27.4 (Pin_4), Q9.3 (D); no longer Q1.3 (D)
- net SD_Detect: no longer names the net of U1.15 (IO3)
- no-connect marks 5 -> 6
Other:
- note removed: "1, 2, 4 for Soil Moisture Sensors"
- note removed: "2 - MOSFET Drain 1 - 12V"
- moved on the sheet: J27

Commit message: added some BOM stuff
Parts:
- C1: footprint (none) -> digikey-footprints:0805; MFG Part Number GRM21BR61E226ME44L -> CL21A226KQCLRNC; Manufacturer (none) -> Samsung Electro-Mechanics; Package (none) -> 0805
- C10, C11, C9: footprint (none) -> digikey-footprints:0805; MFG Part Number (none) -> GRM21BR71C475KE51L; Manufacturer (none) -> Murata Electronics; Package (none) -> 0805 (2012 Metric); Type (SMD/thru-hole, etc.) (none) -> SMD
- C4: value 0.1uF -> 22uF; footprint (none) -> digikey-footprints:0805; MFG Part Number GRM188R71C105KA12D -> CL21A226KQCLRNC; Manufacturer (none) -> Samsung Electro-Mechanics; Package (none) -> 0805; Type (SMD/thru-hole, etc.) (none) -> SMD
- C5, C6: footprint (none) -> digikey-footprints:0805; MFG Part Number (none) -> CL21A226KQCLRNC; Manufacturer (none) -> Samsung Electro-Mechanics; Package (none) -> 0805; Type (SMD/thru-hole, etc.) (none) -> SMD
- J3: Availability Not in stock -> (none); Check_prices https://www.snapeda.com/parts/TYPE-C-31-M-12/HRO+Electronic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 -> (none); Description_1 USB Connectors 24 Receptacle 1 8.94*7.3mm RoHS -> (none); MANUFACTURER HRO Electronics Co., Ltd. -> (none); MAXIMUM_PACKAGE_HEIGHT 3.26 mm -> (none); MF HRO Electronics Co., Ltd. -> (none); MP TYPE-C-31-M-12 -> (none); PARTREV 2020.12.08 -> (none); Package/Footprint Package -> (none); Price None -> (none); SNAPEDA_PN TYPE-C-31-M-12 -> (none); STANDARD Manufacturer Recommendations -> (none); SnapEDA_Link https://www.snapeda.com/parts/TYPE-C-31-M-12/HRO+Electronic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 -> (none)
- U1: Availability Not in stock -> (none); Check_prices https://www.snapeda.com/parts/ESP32-S3-WROOM-1U/Espressif+S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 -> (none); Description_1 2.4 GHz Wi-Fi (802.11 b/g/n) and Bluetooth 5 (LE) module -> (none); MANUFACTURER Espressif -> (none); MAXIMUM_PACKAGE_HEIGHT 3.35mm -> (none); MF Espressif Systems -> (none); MP ESP32-S3-WROOM-1U -> (none); PARTREV v0.6 -> (none); Package/Footprint SMD-41 Espressif Systems -> (none); Price None -> (none); Purchase-URL https://www.snapeda.com/api/url_track_click_mouser/?unipart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 -> (none); STANDARD Manufacturer Recommendations -> (none); SnapEDA_Link https://www.snapeda.com/parts/ESP32-S3-WROOM-1U/Espressif+S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 -> (none)
Connections:
- net 3.3V: now also C11.1; no longer C9.1
- net 5V: now also C9.1; no longer C11.1

Commit message: BOM and footprints
Parts:
- C12, C13, C14, C15, C16, C17, C18, C19, C2, C20, C3, C7, C8, R1, R10, R11, R13, R14, R15, R16, R17, R18, R19, R2, R20, R21, R22, R23, R24, R25, R26, R27, R3, R30, R31, R32, R33, R4, R5, R6, R7, R8, R9: footprint (none) -> digikey-footprints:0805
- D2, D3, D4, D5, D6, D7, D8: footprint (none) -> Diode_SMD:D_SOD-123
- J1: footprint (none) -> TerminalBlock_RND:TerminalBlock_RND_205-00012_1x02_P5.00mm_Horizontal
- J10: footprint (none) -> Connector_Molex:Molex_KK-254_AE-6410-03A_1x03_P2.54mm_Vertical
- J27, SW2: footprint (none) -> Connector_PinHeader_2.54mm:PinHeader_2x13_P2.54mm_Vertical
- J7: footprint (none) -> Connector_Molex:Molex_KK-254_AE-6410-05A_1x05_P2.54mm_Vertical
- JP2, JP3: footprint (none) -> Jumper:SolderJumper-2_P1.3mm_Open_Pad1.0x1.5mm
- L1: footprint (none) -> Inductor_SMD:L_10.4x10.4_H4.8; MFG Part Number (none) -> SMDRH105R-3R3NT; Manufacturer (none) -> SXN(Shun Xiang Nuo Elec); Package (none) -> SMD, 10.4x10.3; Type (SMD/thru-hole, etc.) (none) -> SMD
- MP2393GTL-Z1: footprint (none) -> Package_TO_SOT_SMD:SOT-583-8
- Q1, Q2, Q3, Q4, Q5, Q6, Q7, Q9: footprint (none) -> digikey-footprints:SOT-23-3
- U5: footprint (none) -> digikey-footprints:SOIC-8_W5.3mm
- U6: footprint (none) -> Connector_PinHeader_2.54mm:PinHeader_1x14_P2.54mm_Vertical

Commit message: working on BOM and footprints
Parts:
- removed SW2: Reset, Connector_PinHeader_2.54mm:PinHeader_2x13_P2.54mm_Vertical, symbol Switch:SW_Push
- added SW3: BootMode_Switch, symbol Switch:SW_SPDT
- D2, D3, D4, D5, D6, D7, D8: value 1N4007 -> 1N4007W; MFG Part Number (none) -> 1N4007W; Manufacturer (none) -> FUXINSEMI; Package (none) -> SMD
- J7: footprint Connector_Molex:Molex_KK-254_AE-6410-05A_1x05_P2.54mm_Vertical -> TerminalBlock_RND:TerminalBlock_RND_205-00015_1x05_P5.00mm_Horizontal
- SW5: value BootSwitch -> ResetButton_Internal; footprint (none) -> Button_Switch_SMD:SW_Push_1P1T_XKB_TS-1187A; MFG Part Number (none) -> TS-1187A-B-A-B; Manufacturer (none) -> XKB Connection; Package (none) -> SMD-4P,5.1x5.1mm; Type (SMD/thru-hole, etc.) (none) -> SMD
- U2: footprint (none) -> Package_TO_SOT_SMD:SOT-223-3_TabPin2; MFG Part Number (none) -> MCP1826S-3302E/DB; Manufacturer (none) -> Microchip Tech; Package (none) -> SOT-223-3; Type (SMD/thru-hole, etc.) (none) -> SMD
- U3: footprint (none) -> Package_TO_SOT_SMD:SOT-23-6_Handsoldering; MFG Part Number (none) -> USBLC6-2SC6; Manufacturer (none) -> STMicroelectronics; Package (none) -> SOT-23-6L; Type (SMD/thru-hole, etc.) (none) -> SMD
- U4: value TC4428xOA -> TC4428EOA; footprint (none) -> digikey-footprints:SOIC-8_W3.9mm; MFG Part Number (none) -> TC4428EOA; Manufacturer (none) -> Microchip Tech; Package (none) -> SOIC-8; Type (SMD/thru-hole, etc.) (none) -> SMD
- U5: footprint digikey-footprints:SOIC-8_W5.3mm -> Package_SO:SOIC-8_5.3x5.3mm_P1.27mm; MFG Part Number (none) -> W25Q128JVSIQ; Manufacturer (none) -> Winbond Ele; Package (none) -> SOIC-8 208-mil; Type (SMD/thru-hole, etc.) (none) -> SMD
- U6: MFG Part Number (none) -> NA; Manufacturer (none) -> NA; Package (none) -> pinholes; Type (SMD/thru-hole, etc.) (none) -> Through-hole
Connections:
- net BootMode: now also SW3.3 (C); no longer SW5.1
- net GND: now also SW3.2 (B)
- net Reset_SW renamed Reset_Button
- net Reset_Button: now also SW5.1
- no-connect marks 6 -> 7
Other:
- note added: "GPIO45 held low. Turn on internal pull-up in firmware for fan tach readings"

Commit message: working on stuff
Parts:
- removed SW3: BootMode_Switch, symbol Switch:SW_SPDT
- added SW3: BootMode_Button, Button_Switch_SMD:SW_Push_1P1T_XKB_TS-1187A, symbol Switch:SW_Push
- added USBC1: TYPE-C-31-M-12, easyeda2kicad:USB-C_SMD-TYPE-C-31-M-12_1, symbol easyeda2kicad:TYPE-C-31-M-12
- U1: footprint (none) -> PCM_Espressif:ESP32-S3-WROOM-1U; MFG Part Number (none) -> ESP32-S3-WROOM-1U-N8R8; Manufacturer (none) -> Espressif Systems; Package (none) -> SMD,19.2x18mm; Type (SMD/thru-hole, etc.) (none) -> SMD
Connections:
- net BootMode: now also SW3.1
- net GND: now also SW3.2; no longer U1.41_1 (GND), U1.41_2 (GND), U1.41_3 (GND), U1.41_4 (GND), U1.41_5 (GND), U1.41_6 (GND), U1.41_7 (GND), U1.41_8 (GND), U1.41_9 (GND)
- net MISO: no longer U6.9 (MISO)
- no-connect marks 7 -> 8
Changed lines of the file:
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@@
 	)
 	(no_connect
+		(at 116.84 91.44)
+	)
+	(no_connect
 		(at 195.58 22.86)
 	)
@@
 	(global_label "Gnd"
 		(shape input)
-		(at 16.51 149.86 180)
+		(at 16.51 152.4 180)
 		(fields_autoplaced yes)
 		(effects
@@
 		)
 		(property "Intersheetrefs" "${INTERSHEET_REFS}"
-			(at 9.9568 149.86 0)
+			(at 9.9568 152.4 0)
 			(effects
 				(font
@@
 		)
 	)
-	(global_label "MISO"
-		(shape input)
-		(at 116.84 91.44 0)
-		(fields_autoplaced yes)
-		(effects
-			(font
-				(size 1.27 1.27)
-			)
-			(justify left)
-		)
-		(property "Intersheetrefs" "${INTERSHEET_REFS}"
-			(at 124.4214 91.44 0)
-			(effects
-				(font
-					(size 1.27 1.27)
-				)
-				(justify left)
-				(hide yes)
-			)
-		)
-	)
 	(global_label "SCK"
 		(shape input)
@@
 	)
 	(symbol
+		(lib_id "Switch:SW_Push")
+		(at 21.59 152.4 180)
+		(unit 1)
+		(exclude_from_sim no)
+		(in_bom yes)
+		(on_board yes)
+		(dnp no)
+		(property "Reference" "SW3"
+			(at 21.59 154.94 0)
+			(effects
+				(font
+					(size 1.27 1.27)
+				)
+			)
+		)
+		(property "Value" "BootMode_Button"
+			(at 18.542 149.352 0)
+			(effects
+				(font
+					(size 1.27 1.27)
+				)
+			)
+		)
+		(property "Footprint" "Button_Switch_SMD:SW_Push_1P1T_XKB_TS-1187A"
+			(at 21.59 157.48 0)
+			(effects
+				(font
+					(size 1.27 1.27)
+				)
+				(hide yes)
+			)
+		)
+		(property "Datasheet" "https://jlc-prod-smt.oss-eu-central-1.aliyuncs.com/smtDataManualFile/8550724022091735040-C318884.pdf?response-content-disposition=attachment%3B%20filename%3DC318884.pdf%3B%20filename%2A%3DUTF-8%27%27C318884.pdf&x-oss-date=20260623T203203Z&x-oss-expires=1800&x-oss-security-token=CAISgAN1q6Ft5B2yfSjIr5vsPfTmrKdi%2Ba%2FYOlD8nU0nar5i3fTulTz2IHhMdHJsAOodtv0%2FmmhT6PkclqRLcbhpcmfjV%2BZHzLB8qepJv1ZG4J7b16cNrbH4M4H6aXeirtuwDsz9SNTCALjPD3nPii50x5bjaDymRCbLGJaViJlhHLN1Ow6jdmhpCctxLAlvo9NgFxm3D%2Fu2NQPwiWf9FVdhvhEG6Vly8qOi2MaRmFy8yFTx0b0SvJ%2BjYMrmPctoN9JnSdC5mfdzau3a1TJ84gRD0a5wkaVA1zbDs5bfISEIuUzebreLqY03dV4mOvdqIcMe8qigz88fk%2FfIioH6xyxKOexoSCnFTOiiupCcQLPyao9jLu6iayqViY7QaIOTqQohZmkAMwVOasAsI3Ngh4zF97Qt0cVNkXO9gWfLI8DtuMleWpohUVpD7tHD0eS19jklBdzSlusJRAJJUVBflCeKEaRNSAd3WGhEfM2%2BBt4QT30w5N2u00S8OSMIzGHxnqKWD5sagAGwGdg7eBRMe%2BjpmZKoMN29EbI%2BqeGWDU%2BDN00Al2NVRqyAwYTC2%2BRN3r3KydJAsor2R%2BId%2Fl0%2FMQM8NLpR3Tl%2FttaRfEoqhy9ZHOrBuuyJcP8ULoQ3qLZ6xiB%2FQQRtxnhSFSTuxrRbCzjPg0RpjFkz%2FPFgFCM03kfF1QwKI%2FFgsCAA&x-oss-signature-version=OSS4-HMAC-SHA256&x-oss-credential=STS.NXYvNRAxCNm38vMyMrf1N21Ew%2F20260623%2Feu-central-1%2Foss%2Faliyun_v4_request&x-oss-signature=e43aa02dab2f35991183760960ab48201f603011864f04475b1513b165997cdf"
+			(at 21.59 157.48 0)
+			(effects
+				(font
+					(size 1.27 1.27)
+				)
+				(hide yes)
+			)
+		)
+		(property "Description" "Push button switch, generic, two pins"
+			(at 21.59 152.4 0)
+			(effects
+				(font
+					(size 1.27 1.27)
+				)
+				(hide yes)
+			)
+		)
+		(property "MFG Part Number" "TS-1187A-B-A-B "
+			(at 21.59 152.4 0)
+			(effects
+				(font
+					(size 1.27 1.27)
+				)
+				(hide yes)
+			)
+		)
+		(property "Type (SMD/thru-hole, etc.)" "SMD"
+			(at 21.59 152.4 0)
+			(effects
+				(font
+					(size 1.27 1.27)
+				)
+				(hide yes)
+			)
+		)
+		(property "Manufacturer" "XKB Connection"
+			(at 21.59 152.4 0)
+			(effects
+				(font
+					(size 1.27 1.27)
+				)
+				(hide yes)
+			)
+		)
+		(property "Package" "SMD-4P,5.1x5.1mm "
+			(at 21.59 152.4 0)
+			(effects
+				(font
+					(size 1.27 1.27)
+				)
+				(hide yes)
+			)
+		)
+		(pin "2"
+		)
+		(pin "1"
+		)
+		(instances
+			(project "GrowChamberPCB"
+				(path "/39371779-5336-4073-adec-fb32caf6a86f"
+					(reference "SW3")
+					(unit 1)
+				)
+			)
+		)
+	)
+	(symbol
 		(lib_id "Device:R")
 		(at 69.85 39.37 180)
@@
 			)
 		)
-		(property "Footprint" ""
+		(property "Footprint" "PCM_Espressif:ESP32-S3-WROOM-1U"
 			(at 67.31 165.1 0)
 			(effects
@@
 			)
 		)
-		(property "Description" ""
+		(property "Description" "microcontroller"
 			(at 67.31 165.1 0)
 			(effects
@@
 			)
 		)
-		(property "MFG Part Number" ""
+		(property "MFG Part Number" "ESP32-S3-WROOM-1U-N8R8 "
 			(at 67.31 165.1 0)
 			(effects
@@
 			)
 		)
-		(property "Type (SMD/thru-hole, etc.)" ""
+		(property "Type (SMD/thru-hole, etc.)" "SMD"
 			(at 67.31 165.1 0)
 			(effects
@@
 			)
 		)
-		(property "Manufacturer" ""
+		(property "Manufacturer" "Espressif Systems"
 			(at 67.31 165.1 0)
 			(effects
@@
 			)
 		)
-		(property "Package" ""
+		(property "Package" "SMD,19.2x18mm"
 			(at 67.31 165.1 0)
 			(effects
@@
 		(pin "1"
 		)
-		(pin "41_3"
-		)
-		(pin "41_2"
-		)
-		(pin "41_6"
-		)
 		(pin "34"
 		)
 		(pin "25"
 		)
-		(pin "41_4"
-		)
 		(pin "24"
 		)
-		(pin "41_8"
-		)
 		(pin "33"
 		)
@@
 		(pin "40"
 		)
-		(pin "41_5"
-		)
 		(pin "32"
 		)
-		(pin "41_7"
-		)
 		(pin "35"
 		)
-		(pin "41_9"
-		)
 		(pin "26"
 		)
-		(pin "41_1"
-		)
 		(instances
 			(project "GrowChamberPCB"
@@
 	)
 	(symbol
+		(lib_id "easyeda2kicad:TYPE-C-31-M-12")
+		(at 173.99 -13.97 0)
+		(unit 1)
+		(exclude_from_sim no)
+		(in_bom yes)
+		(on_board yes)
+		(dnp no)
+		(fields_autoplaced yes)
+		(property "Reference" "USBC1"
+			(at 176.53 -34.29 0)
+			(effects
+				(font
+					(size 1.27 1.27)
+				)
+			)
+		)
+		(property "Value" "TYPE-C-31-M-12"
+			(at 176.53 -31.75 0)
+			(effects
+				(font
+					(size 1.27 1.27)
+				)
+			)
+		)
+		(property "Footprint" "easyeda2kicad:USB-C_SMD-TYPE-C-31-M-12_1"
+			(at 173.99 7.62 0)
+			(effects
+				(font
+					(size 1.27 1.27)
+				)
+				(hide yes)
+			)
+		)
+		(property "Datasheet" "https://lcsc.com/product-detail/USB-Type-C_Korean-Hroparts-Elec-TYPE-C-31-M-12_C165948.html"
+			(at 173.99 10.16 0)
+			(effects
+				(font
+					(size 1.27 1.27)
+				)
+				(hide yes)
+			)
+		)
+		(property "Description" ""
+			(at 173.99 -13.97 0)
+			(effects
+				(font
+					(size 1.27 1.27)
+				)
+				(hide yes)
+			)
+		)
+		(property "Manufacturer" "韩国韩荣"
+			(at 173.99 12.7 0)
+			(effects
+				(font
+					(size 1.27 1.27)
+				)
+				(hide yes)
+			)
+		)
+		(property "MPN" "TYPE-C-31-M-12"
+			(at 173.99 15.24 0)
+			(effects
+				(font
+					(size 1.27 1.27)
+				)
+				(hide yes)
+			)
+		)
+		(property "LCSC Part" "C165948"
+			(at 173.99 17.78 0)
+			(effects
+				(font
+					(size 1.27 1.27)
+				)
+				(hide yes)
+			)
+		)
+		(pin "B4A9"
+		)
+		(pin "1"
+		)
+		(pin "A8"
+		)
+		(pin "2"
+		)
+		(pin "B1A12"
+		)
+		(pin "B5"
+		)
+		(pin "4"
+		)
+		(pin "B6"
+		)
+		(pin "A4B9"
+		)
+		(pin "A1B12"
+		)
+		(pin "B8"
+		)
+		(pin "A6"
+		)
+		(pin "B7"
+		)
+		(pin "A5"
+		)
+		(pin "3"
+		)
+		(pin "A7"
+		)
+		(instances
+			(project "GrowChamberPCB"
+				(path "/39371779-5336-4073-adec-fb32caf6a86f"
+					(reference "USBC1")
+					(unit 1)
+				)
+			)
+		)
+	)
+	(symbol
 		(lib_id "Device:C")
 		(at 48.26 137.16 90)
@@
 					(unit 1)
 				)
-			)
-		)
-	)
-	(symbol
-		(lib_id "Switch:SW_SPDT")
-		(at 21.59 149.86 0)
-		(unit 1)
-		(exclude_from_sim no)
-		(in_bom yes)
-		(on_board yes)
-		(dnp no)
-		(property "Reference" "SW3"
-			(at 17.78 144.526 0)
-			(effects
-				(font
-					(size 1.27 1.27)
-				)
-			)
-		)
-		(property "Value" "BootMode_Switch"
-			(at 21.59 144.018 0)
-			(effects
-				(font
-					(size 1.27 1.27)
-				)
-			)
-		)
-		(property "Footprint" ""
-			(at 21.59 149.86 0)
-			(effects
-				(font
-					(size 1.27 1.27)
-				)
-				(hide yes)
-			)
-		)
-		(property "Datasheet" "~"
-			(at 21.59 157.48 0)
-			(effects
-				(font
-					(size 1.27 1.27)
-				)
-				(hide yes)
-			)
-		)
-		(property "Description" "Switch, single pole double throw"
-			(at 21.59 149.86 0)
-			(effects
-				(font
-					(size 1.27 1.27)
-				)
-				(hide yes)
-			)
-		)
-		(property "MFG Part Number" ""
-			(at 21.59 149.86 0)
-			(effects
-				(font
-					(size 1.27 1.27)
-				)
-				(hide yes)
-			)
-		)
-		(pin "1"
-		)
-		(pin "3"
-		)
-		(pin "2"
-		)
-		(instances
-			(project "GrowChamberPCB"
-				(path "/39371779-5336-4073-adec-fb32caf6a86f"
-					(reference "SW3")
-					(unit 1)
-				)
