File: GrowChamberPCB/GrowChamberPCB.kicad_sch (KiCad schematic)
At the start: 5 parts, among them CN2 RelayBoard Interconnect, P1 To Faceplate, U4 To Faceplate, U6 CR2013-MI2120

Commit message: almost done!
Parts:
- removed P1: To Faceplate, easyeda2kicad:CONN-TH_3P-P5.00_WJ127-5.0-3P, symbol easyeda2kicad:WJ127-5.0-3P
- added 12V_IN4, LED_To_Connector1: Screw Terminal, easyeda2kicad:CONN-TH_2P-P5.00_CPC3703CTR, symbol easyeda2kicad:WJ127-5.0-2P
- added D4: SD15, easyeda2kicad:SOD-323_L1.7-W1.3-LS2.6-RD, symbol easyeda2kicad:SD15_C2931147
- renumbered 12V_IN to 12V_IN1
Connections:
- net Gnd is gone; now on net GND: U6.2 (GND)
- net 12V: now also 12V_IN4.2, LED_To_Connector1.1
- net GND: now also 12V_IN4.1
- net LEDs: now also U4.24, D4.1 (C), LED_To_Connector1.2
- new net GND_FP: D4.2 (A)
- no-connect marks 2 -> 3
Other:
- moved on the sheet: U6

Commit message: more pcb
Parts:
- P1: renamed from 12V_IN1; value Screw Terminal -> 12V_In
Changed lines of the file:
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@@
 		(dnp no)
 		(fields_autoplaced yes)
-		(property "Reference" "12V_IN1"
-			(at 269.24 20.32 90)
+		(property "Reference" "P1"
+			(at 265.43 19.0499 0)
 			(effects
 				(font
 					(size 1.27 1.27)
 				)
+				(justify left)
 			)
 		)
-		(property "Value" "Screw Terminal"
-			(at 266.7 20.32 90)
+		(property "Value" "12V_In"
+			(at 265.43 21.5899 0)
 			(effects
 				(font
 					(size 1.27 1.27)
 				)
+				(justify left)
 			)
 		)
@@
 			(project "GrowChamberPCB"
 				(path "/e884bae1-e2d9-44d2-8169-161aa31a84ae"
-					(reference "12V_IN1")
+					(reference "P1")
 					(unit 1)
 				)
