File: GrowChamberPCB/ESP32.kicad_sch (KiCad schematic)
At the start: 50 parts, among them J42 TP, J43 TP, J44 TP, J45 TP, J47 Conn_01x04, J48 Conn_01x09, SW1 Reset_Button_Internal, SW3 Bootmode_Internal, U3 ESP32-S3-WROOM-1U-N8R8, U7 TC4428EOA, U8 Memory

Commit message: finished routing
Parts:
- removed C12, C13: 22uF X7R, easyeda2kicad:C1206, symbol easyeda2kicad:TCC1206X5R226K250HT
- removed C14: 1uF, easyeda2kicad:C0603, symbol easyeda2kicad:CL10B105KA8NNNC
- removed C15: 0.1nF, easyeda2kicad:C0603, symbol easyeda2kicad:CL10B104KB8NNNC
- removed C18: 100nF, easyeda2kicad:C0603, symbol easyeda2kicad:CL10B104KO8NNNC
- removed C19: 10uF, easyeda2kicad:C0603, symbol easyeda2kicad:CL10A106KO8NQNC
- removed D1, D18, D3: SRV05-4_C2836319, easyeda2kicad:SOT-23-6_L2.9-W1.6-P0.95-LS2.8-BL, symbol easyeda2kicad:SRV05-4_C2836319
- removed D19: USBLC6-2SC6, easyeda2kicad:SOT-23-6_L2.9-W1.6-P0.95-LS2.8-BL, symbol easyeda2kicad:USBLC6-2SC6
- removed R10, R11, R15, R48, R49, R50, R6, R7: 10K, easyeda2kicad:R0603, symbol easyeda2kicad:AC0603FR-0710KL
- removed R12, R13: 5.1k, easyeda2kicad:R0603, symbol easyeda2kicad:AC0603FR-075K1L
- removed R43, R5, R54, R55, R56, R57, R58, R59: 33, easyeda2kicad:R0603, symbol easyeda2kicad:RS-03K33R0FT
- removed R46, R47: 100K, easyeda2kicad:R0603, symbol easyeda2kicad:RT0603BRD07100KL
- removed R51, R60: 1k, easyeda2kicad:R0603, symbol easyeda2kicad:FRC0603J102TS
- removed R8, R9: 22, easyeda2kicad:R0603, symbol easyeda2kicad:RT0603BRD0710KL
- removed SW1: Reset_Button_Internal, easyeda2kicad:SW-SMD_L4.0-W2.9-LS5.0, symbol easyeda2kicad:HXTS-1088-AR02016
- added C10: 22uF - X5R, easyeda2kicad:C1206, symbol easyeda2kicad:CL31A226KAHNNNE
- added C13: 4.7uF - X7R, easyeda2kicad:C1206, symbol easyeda2kicad:1206B475K500NT
- added C14: 150pF, easyeda2kicad:C0603, symbol easyeda2kicad:0603B151K500NT
- added C15, C5: 100nF, easyeda2kicad:C0402, symbol easyeda2kicad:CL05B104KO5NNNC
- added C6: 10uF, easyeda2kicad:C0805, symbol easyeda2kicad:CL21A106KAYNNNE
- added H1, H2, H3, H4: MountingHole, MountingHole:MountingHole_3.2mm_M3_Pad_Via, symbol Mechanical:MountingHole
- added R10, R21: 1k, easyeda2kicad:R0603, symbol easyeda2kicad:0603WAF1001T5E
- added R11, R12, R13, R15, R29, R43, R46, R7, R9: 33, easyeda2kicad:R0603, symbol easyeda2kicad:0603WAF330JT5E
- added R14, R17, R24, R25, R26, R27, R28, R30: 10k, easyeda2kicad:R0603, symbol easyeda2kicad:0603WAF1002T5E
- added R19, R20: 100k, easyeda2kicad:R0603, symbol easyeda2kicad:0603WAF1003T5E
- added R22, R23: 5.1k, easyeda2kicad:R0603, symbol easyeda2kicad:0603WAF5101T5E
- added R6, R8: 22, easyeda2kicad:R0603, symbol easyeda2kicad:0603WAF220JT5E
- added SW1: TS-1088-AR02016, easyeda2kicad:SW-SMD_L3.9-W3.0-P4.45, symbol easyeda2kicad:TS-1088-AR02016
- C16, C17, J42, J43, J44, J45: now in the parts list
- J47, J48: KiLib_Generator (none) -> connector/pin_header_socket; now in the parts list
- LED13, SW3: now not fitted
Connections:
- net Out_D+ is gone; now on net D+: C16.1
- net Out_D- is gone; now on net D-: C17.1
- net 12V: now also C5.2, C6.2, R21.2
- net 3.3V: now also C10.1, C15.1, R24.1, R25.1, R26.2, R27.1, R28.2, R30.2
- net CS_Display: now also R46.1
- net CS_Memory: now also R43.1
- net CS_SD: now also R11.1
- net CircFan_IO: now also U3.4 (IO4); no longer U3.18 (IO10)
- net D+: now also R8.1
- net D-: now also R6.1
- net DC_Display: now also U3.10 (IO17); no longer U3.7 (IO7)
- net Display_Reset: now also U3.11 (IO18); no longer U3.6 (IO6)
- net DrainLevel_IO: now also R14.2, R19.2
- net DrainSolIO: now also U3.18 (IO10); no longer U3.4 (IO4)
- net Drain_Level: now also R14.1
- net EN: now also C13.2, C14.1, R25.2, SW1.2
- net External_Fan_PWM: now also R10.2
- net Fan_Tach: now also U3.38 (IO2); no longer U3.39 (IO1)
- net FloatSwitch_IO: now also R17.2, R20.2
- net FoggerSol_IO: now also U3.17 (IO9); no longer U3.19 (IO11)
- net Fogger_Basin_Float_Switch: now also R17.1
- net GND: now also C10.2, C13.1, C14.2, C15.2, C5.1, C6.1, R19.1, R20.1, R22.2, R23.2, SW1.1
- net GlycolSol_IO: now also U3.19 (IO11); no longer U3.17 (IO9)
- net HeaterFans_IO: now also U3.16 (IO46); no longer U3.20 (IO12)
- net IO19: now also R6.2
- net IO20: now also R8.2
- net MISO: now also U3.7 (IO7), R15.2, R29.2; no longer J47.3 (Pin_3), U8.2 (DO)
- net MOSI: now also R13.1
- net RXD0: now also R7.2
- net SCK: now also R12.1
- net SCL: now also U3.32 (IO39), R28.1; no longer U3.26 (IO45)
- net SDA: now also U3.33 (IO40), R30.1; no longer U3.25 (IO48)
- net Soil_Moisture1: now also U3.26 (IO45); no longer U3.33 (IO40)
- net Soil_Moisture2: now also U3.25 (IO48); no longer U3.32 (IO39)
- net TXD0: now also R9.2
- net WaterSol_IO: now also U3.20 (IO12); no longer U3.16 (IO46)
- net at USB1.B5 (CC2): now also R23.1
- net at SW3.1: now also R24.2
- net at USB1.A5 (CC1): now also R22.1
- net at LED13.2 (A): now also R21.1
- net at U3.37 (TXD0): now also R9.1
- net at U3.12 (IO8): now also R46.2
- net at U3.9 (IO16): now also R11.2
- net Heartbeat_LED: now reaches U3.15 (IO3)
- net at U3.36 (RXD0): now also R7.1
- net at U3.5 (IO5): now also R12.2
- net at U3.8 (IO15): now also R43.2
- net at U8.3 (IO2): now also R27.2
- net at U8.7 (IO3): now also R26.1
- new net: R10.1, U3.39 (IO1)
- new net: R13.2, U3.6 (IO6)
- new net: R15.1, U8.2 (DO)
- new net MISO_ESD: J47.3 (Pin_3), R29.1
- no-connect marks 13 -> 15
Other:
- added sheet Data Line ESD (3.3VESD.kicad_sch)
- added sheet Data Line ESD1 (3.3VESD.kicad_sch)
- added sheet Data Line ESD2 (3.3VESD.kicad_sch)
- added sheet Data Line ESD3 (3.3VESD.kicad_sch)

Commit message: fixing stuff
Parts:
- U3: now not fitted
Other:
- sheet Data Line ESD ports: added GND, Power; removed none
- sheet Data Line ESD1 ports: added GND, Power; removed none
- sheet Data Line ESD2 ports: added GND, Power; removed none
- sheet Data Line ESD3 ports: added GND, Power; removed none

Commit message: started box
Parts:
- removed C16, C17: DNP, easyeda2kicad:C1206, symbol easyeda2kicad:TCC1206X5R226K250HT
- removed R14, R17, R24, R25, R26, R27, R28, R30: 10k, easyeda2kicad:R0603, symbol easyeda2kicad:0603WAF1002T5E
- removed U7: TC4428EOA, easyeda2kicad:SOIC-8_L4.9-W3.9-P1.27-LS6.0-BL, symbol easyeda2kicad:TC4428EOA
- added R53, R54, R55, R56, R57, R59, R61: 10K, easyeda2kicad:R0805, symbol easyeda2kicad:0805W8F1002T5E
- added U1: TC4428EOA713-TUDI, easyeda2kicad:SOIC-8_L4.9-W3.9-P1.27-LS6.0-BL, symbol easyeda2kicad:TC4428EOA713-TUDI
Connections:
- net 12V: now also U1.2 (INA)
- net 3.3V: now also R53.2, R54.1, R55.2, R56.2, R57.2
- net DrainLevel_IO: now also R61.1
- net Drain_Level: now also R61.2
- net EN: now also R54.2
- net FloatSwitch_IO: now also R59.1
- net Fogger_Basin_Float_Switch: now also R59.2
- net Fogger_PWM: now also U1.6 (VDD), U1.8 (NC)
- net GND: now also U1.7 (~{OUTA})
- net Piezo1: now also U1.1 (NC)
- net Piezo2: now also U1.3 (GND)
- net SCL: now also R56.1
- net SDA: now also R55.1
- net Memory_IO3: now reaches U8.3 (IO2)
- net Memory_IO3: now also U8.7 (IO3), R57.1
- net at SW3.1: now also R53.1
