File: GrowChamberPCB/Faceplate.kicad_sch (KiCad schematic)
At the start: 56 parts, among them J1 Mister, J10 FoggerBasin, J12 Moisture Sensor 3, J13 Moisture Sensor 2, J14 UART, J15 FAE Fan, J16 DrainLevel, J2 Moisture Sensor 1, J3 SCD30, J4 Heater Fans, J49 TP, J5 Fogger Solenoid, J50 TP, J6 Drain Solenoid, J7 Water Solenoid, J8 Glycol Solenoid, J9 CircFan, SW2 ResetButton_External, SW4 BootMode_External, U2 ZX-IDC2.54-2-13PZZ, U20 PCA9555APW,118

Commit message: finished routing
Parts:
- removed D10, D11, D12, D14, D15, D5, D6, D7, D8, D9: SD15, easyeda2kicad:SOD-323_L1.7-W1.3-LS2.6-RD, symbol easyeda2kicad:SD15_C2931147
- removed LED11: FAE, easyeda2kicad:LED-TH_BD3.9-P2.54-RD_RED, symbol easyeda2kicad:EL304RD
- removed LED12: LED On, easyeda2kicad:LED-TH_BD3.9-P2.54-RD_RED, symbol easyeda2kicad:EL304RD
- removed R29, R31, R35: 75, easyeda2kicad:R0603, symbol easyeda2kicad:RS-03K75R0FT
- removed R33, R36, R37, R38, R39, R40, R41, R42, R44: 1k, easyeda2kicad:R0603, symbol easyeda2kicad:FRC0603J102TS
- removed SW2: ResetButton_External, easyeda2kicad:CONN-TH_PB-05B-R, symbol easyeda2kicad:PB-05B-R
- removed U20: PCA9555APW,118, easyeda2kicad:TSSOP-24_L7.8-W4.4-P0.65-LS6.4-BL, symbol easyeda2kicad:PCA9555APW,118
- added D1, D10, D11, D12, D3, D5, D6, D7, D8, D9: SMF15A, easyeda2kicad:SOD-123FL_L2.7-W1.8-LS3.8-RD, symbol easyeda2kicad:SMF15A_C19077509
- added H5, H6: MountingHole, MountingHole:MountingHole_3.2mm_M3_Pad_Via, symbol Mechanical:MountingHole
- added J60: TP, TestPoint:TestPoint_Pad_D2.0mm, symbol Connector_Generic:Conn_01x01
- added R16, R18, R32, R33, R34, R35, R37, R38, R39: 1k, easyeda2kicad:R0603, symbol easyeda2kicad:0603WAF1001T5E
- added R31: 10k, easyeda2kicad:R0603, symbol easyeda2kicad:0603WAF1002T5E
- added R36: 0603WAF750JT5E, easyeda2kicad:R0603, symbol easyeda2kicad:0603WAF750JT5E
- added SW5: On/Off, easyeda2kicad:SW-TH_SS-12D02-VG4, symbol easyeda2kicad:SS-12D02-VG4
- J1, J10, J12, J13, J14, J15, J16, J2, J3, J4, J5, J6, J7, J8, J9: now in the parts list
- J49: value TP -> 12V; now in the parts list
- J50: value TP -> Gnd; now in the parts list
- LED1, LED2, LED3, LED8, LED9, Power_FP1, SW4: now not fitted
- LED10: value Mister -> 12V On; now not fitted
- LED4: value Glycol Solenoid -> 12V On; now not fitted
- LED5: value Water Solenoid -> 12V On; now not fitted
- LED6: value Drain Solenoid -> 12V On; now not fitted
- LED7: value Fogger Solenoid -> 12V On; now not fitted
- U2: value ZX-IDC2.54-2-13PZZ -> 2x13; now not fitted
Connections:
- net 12V_FP: now also R16.2, R18.2, R32.2, R33.2, R34.2, R35.2, R37.2, R38.2, R39.2
- net 3.3V_FP: now also J16.2 (Pin_2), U2.18, U2.20, J60.1 (Pin_1); no longer J16.1 (Pin_1), U2.2, U2.4
- net Circ_Fan_FP: now also U2.24, D5.1 (K); no longer U2.19
- net DrainSol_FP: now also LED5.1 (K), U2.19, D10.1 (K); no longer LED6.1 (K), U2.17
- net Drain_Level_FP: now also J16.1 (Pin_1), U2.6; no longer J16.2 (Pin_2), U2.16
- net EN_FP: now also U2.2, SW5.2; no longer U2.6
- net External_Fan_PWM_FP: now also U2.25, D1.1 (K); no longer U2.24
- net Fan_Tach_FP: now also U2.23, D3.1 (K); no longer U2.26
- net FoggerSol_FP: now also J7.1 (Pin_1), LED4.1 (K), U2.21, D11.1 (K); no longer J5.1 (Pin_1), LED7.1 (K), U2.13
- net Fogger_Basin_Float_Switch_FP: now also U2.4; no longer U2.18
- net GND_FP: now also D1.2 (A), D10.2 (A), D11.2 (A), D12.2 (A), D3.2 (A), D5.2 (A), D6.2 (A), D7.2 (A), D8.2 (A), D9.2 (A), R36.2, SW5.3
- net GlycolSol_FP: now also LED10.1 (K), U2.17, D12.1 (K); no longer LED4.1 (K), U2.11
- net Heater Fans_FP: now also U2.22, D8.1 (K); no longer U2.15
- net Heater_ON_FP: now also U2.1; no longer U2.5
- net LEDs_FP: now also U2.3; no longer U2.7
- net Piezo1_FP: now also J1.2 (Pin_2), U2.7, D7.1 (K); no longer J1.1 (Pin_1), U2.3
- net Piezo2_FP: now also J1.1 (Pin_1), U2.5, D6.1 (K); no longer J1.2 (Pin_2), U2.1
- net RXD0_FP: now also U2.10; no longer U2.20
- net SCL_FP: now also U2.11; no longer U2.25
- net SDA_FP: now also U2.12; no longer U2.23
- net SoilMoisture2_FP: now also U2.15; no longer U2.12
- net SoilMoisture4_FP: now also U2.13; no longer U2.10
- net TXD0_FP: now also U2.9; no longer U2.22
- net WaterSol_FP: now also J5.1 (Pin_1), LED6.1 (K), U2.16, D9.1 (K); no longer J7.1 (Pin_1), LED5.1 (K), U2.9
- net at LED2.2 (A): now also R18.1
- net at LED4.2 (A): now also R33.1
- net at LED9.2 (A): now also R39.1
- net at LED5.2 (A): now also R34.1
- net at LED10.2 (A): now also R37.1
- net at LED6.2 (A): now also R35.1
- net at LED3.2 (A): now also R32.1
- net Heartbeat_LED_FP: now reaches LED7.2 (A)
- net Heartbeat_LED_FP: now also U2.26
- net at LED8.2 (A): now also R38.1
- net at SW4.1: now also R31.2
- net at LED1.2 (A): now also R16.1
- new net: LED7.1 (K), R36.1
- new net 3.3V: R31.1
- no-connect marks 19 -> 3
Other:
- added sheet Data Line ESD1 (3.3VESD.kicad_sch)

Commit message: fixing stuff
Other:
- sheet 3.3V ESD ports: added GND, Power; removed none
- sheet 3.3V ESD2 ports: added GND, Power; removed none
- sheet Data Line ESD ports: added GND, Power; removed none
- sheet Data Line ESD1 ports: added GND, Power; removed none

Commit message: started box
Parts:
- removed R31: 10k, easyeda2kicad:R0603, symbol easyeda2kicad:0603WAF1002T5E
- added R63: 10K, easyeda2kicad:R0805, symbol easyeda2kicad:0805W8F1002T5E
Connections:
- net 3.3V_FP: now also R63.2
- net at SW4.1: now also R63.1
Changed lines of the file:
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@@
 		)
 	)
+	(global_label "3.3V_FP"
+		(shape input)
+		(at 13.97 30.48 180)
+		(fields_autoplaced yes)
+		(effects
+			(font
+				(size 1.27 1.27)
+			)
+			(justify right)
+		)
+		(property "Intersheetrefs" "${INTERSHEET_REFS}"
+			(at 3.5462 30.48 0)
+			(hide yes)
+			(show_name no)
+			(do_not_autoplace no)
+			(effects
+				(font
+					(size 1.27 1.27)
+				)
+				(justify right)
+			)
+		)
+	)
 	(global_label "SCL_FP"
 		(shape input)
@@
 		)
 	)
-	(global_label "3.3V"
-		(shape input)
-		(at 13.97 30.48 180)
-		(fields_autoplaced yes)
-		(effects
-			(font
-				(size 1.27 1.27)
-			)
-			(justify right)
-		)
-		(property "Intersheetrefs" "${INTERSHEET_REFS}"
-			(at 6.8724 30.48 0)
-			(hide yes)
-			(show_name no)
-			(do_not_autoplace no)
-			(effects
-				(font
-					(size 1.27 1.27)
-				)
-				(justify right)
-			)
-		)
-	)
 	(global_label "3.3V_FP"
 		(shape input)
@@
 	)
 	(symbol
-		(lib_id "easyeda2kicad:0603WAF1002T5E")
-		(at 19.05 30.48 0)
-		(unit 1)
-		(body_style 1)
-		(exclude_from_sim no)
-		(in_bom yes)
-		(on_board yes)
-		(in_pos_files yes)
-		(dnp no)
-		(property "Reference" "R31"
-			(at 19.558 32.512 0)
-			(show_name no)
-			(do_not_autoplace no)
-			(effects
-				(font
-					(size 1.27 1.27)
-				)
-			)
-		)
-		(property "Value" "10k"
-			(at 19.304 27.94 0)
-			(show_name no)
-			(do_not_autoplace no)
-			(effects
-				(font
-					(size 1.27 1.27)
-				)
-			)
-		)
-		(property "Footprint" "easyeda2kicad:R0603"
-			(at 19.05 38.1 0)
-			(hide yes)
-			(show_name no)
-			(do_not_autoplace no)
-			(effects
-				(font
-					(size 1.27 1.27)
-				)
-			)
-		)
-		(property "Datasheet" "https://lcsc.com/product-detail/Chip-Resistor-Surface-Mount-UniOhm_10KR-1002-1_C25804.html"
-			(at 19.05 40.64 0)
-			(hide yes)
-			(show_name no)
-			(do_not_autoplace no)
-			(effects
-				(font
-					(size 1.27 1.27)
-				)
-			)
-		)
-		(property "Description" "10KΩ (1002) ±1%"
-			(at 19.05 30.48 0)
-			(hide yes)
-			(show_name no)
-			(do_not_autoplace no)
-			(effects
-				(font
-					(size 1.27 1.27)
-				)
-			)
-		)
-		(property "Manufacturer" "UNI-ROYAL(厚声)"
-			(at 19.05 43.18 0)
-			(hide yes)
-			(show_name no)
-			(do_not_autoplace no)
-			(effects
-				(font
-					(size 1.27 1.27)
-				)
-			)
-		)
-		(property "MPN" "0603WAF1002T5E"
-			(at 19.05 45.72 0)
-			(hide yes)
-			(show_name no)
-			(do_not_autoplace no)
-			(effects
-				(font
-					(size 1.27 1.27)
-				)
-			)
-		)
-		(property "LCSC Part" "C25804"
-			(at 19.05 48.26 0)
-			(hide yes)
-			(show_name no)
-			(do_not_autoplace no)
-			(effects
-				(font
-					(size 1.27 1.27)
-				)
-			)
-		)
-		(pin "2"
-		)
-		(pin "1"
-		)
-		(instances
-			(project "GrowChamberPCB"
-				(path "/e884bae1-e2d9-44d2-8169-161aa31a84ae/c2403359-39ea-416b-9a92-81a595d10d09"
-					(reference "R31")
-					(unit 1)
-				)
-			)
-		)
-	)
-	(symbol
 		(lib_id "easyeda2kicad:WJ127-5.0-2P")
 		(at 191.77 25.4 0)
@@
 					(unit 1)
 				)
+			)
+		)
+	)
+	(symbol
+		(lib_id "easyeda2kicad:0805W8F1002T5E")
+		(at 19.05 30.48 180)
+		(unit 1)
+		(body_style 1)
+		(exclude_from_sim no)
+		(in_bom yes)
+		(on_board yes)
+		(in_pos_files yes)
+		(dnp no)
+		(fields_autoplaced yes)
+		(property "Reference" "R63"
+			(at 19.05 24.13 0)
+			(show_name no)
+			(do_not_autoplace no)
+			(effects
+				(font
+					(size 1.27 1.27)
+				)
+			)
+		)
+		(property "Value" "10K"
+			(at 19.05 26.67 0)
+			(show_name no)
+			(do_not_autoplace no)
+			(effects
+				(font
+					(size 1.27 1.27)
+				)
+			)
+		)
+		(property "Footprint" "easyeda2kicad:R0805"
+			(at 19.05 22.86 0)
+			(hide yes)
+			(show_name no)
+			(do_not_autoplace no)
+			(effects
+				(font
+					(size 1.27 1.27)
+				)
+			)
+		)
+		(property "Datasheet" "https://lcsc.com/product-detail/Chip-Resistor-Surface-Mount-UniOhm_10KR-1002-1_C17414.html"
+			(at 19.05 20.32 0)
+			(hide yes)
+			(show_name no)
+			(do_not_autoplace no)
+			(effects
+				(font
+					(size 1.27 1.27)
+				)
+			)
+		)
+		(property "Description" "10KΩ (1002) ±1%"
+			(at 19.05 30.48 0)
+			(hide yes)
+			(show_name no)
+			(do_not_autoplace no)
+			(effects
+				(font
+					(size 1.27 1.27)
+				)
+			)
+		)
+		(property "Manufacturer" "UNI-ROYAL(厚声)"
+			(at 19.05 17.78 0)
+			(hide yes)
+			(show_name no)
+			(do_not_autoplace no)
+			(effects
+				(font
+					(size 1.27 1.27)
+				)
+			)
+		)
+		(property "MPN" "0805W8F1002T5E"
+			(at 19.05 15.24 0)
+			(hide yes)
+			(show_name no)
+			(do_not_autoplace no)
+			(effects
+				(font
+					(size 1.27 1.27)
+				)
+			)
+		)
+		(property "LCSC Part" "C17414"
+			(at 19.05 12.7 0)
+			(hide yes)
+			(show_name no)
+			(do_not_autoplace no)
+			(effects
+				(font
+					(size 1.27 1.27)
+				)
+			)
+		)
+		(pin "2"
+		)
+		(pin "1"
+		)
+		(instances
+			(project "GrowChamberPCB"
+				(path "/e884bae1-e2d9-44d2-8169-161aa31a84ae/c2403359-39ea-416b-9a92-81a595d10d09"
+					(reference "R63")
+					(unit 1)
+				)
