File: GrowChamberPCB/GrowChamberPCB.kicad_pcb (KiCad board)
At the start: 2 copper layers, 191.2 x 138.5 mm, 158 parts, among them CN2 RelayBoard Interconnect, CN3 Connector_RB, J1 Conn_01x02_Pin, J10 Conn_01x02_Pin, J12 Conn_01x03_Pin, J13 Conn_01x03_Pin, J14 Conn_01x03_Pin, J15 Conn_01x04_Pin, J16 Conn_01x02_Pin, J2 Conn_01x03_Pin, J3 Conn_01x04_Pin, J4 Conn_01x02_Pin, J5 Conn_01x02_Pin, J6 Conn_01x02_Pin, J7 Conn_01x02_Pin, J8 Conn_01x02_Pin, J9 Conn_01x02_Pin, K1 G5LE-14 DC12, Q1 AO3400A_C347475, Q10 NPN, Q11 AO3400A_C347475, Q12 NPN, Q13 AO3400A_C347475, Q14 NPN, Q15 NPN, Q16 AO3400A_C347475, Q2 NPN, Q3 AO3400A_C347475, Q4 NPN, Q5 AO3400A_C347475, Q6 NPN, Q7 AO3400A_C347475, Q8 BRT30N70P3, Q9 NPN, SW1 Reset_Button_Internal, SW2 ResetButton_External, SW3 Bootmode_Internal, SW4 BootMode_External, U1 MP2393GTL-Z, U10 ACS712ELCTR-05B-T, U11 1N4007W, U12 1N4007W, U13 1N4007W, U14 1N4007W, U15 1N4007W, U16 1N4007W, U17 1N4007W, U19 To Faceplate, U2 MCP1826S-3302E/DB, U20 PCA9555APW,118, U3 ESP32-S3-WROOM-1U-N8R8, U4 To Faceplate, U5 1N4007W, U6 CR2013-MI2120, U7 TC4428EOA, U8 W25Q128JVSIQTR, U9 1N4007W

Commit message: more pcb
Parts:
- removed ?: , 
- added D14: SD15, easyeda2kicad:SOD-323_L1.7-W1.3-LS2.6-RD, F.Cu at (271.2, 73.9)
- added D15: SD15, easyeda2kicad:SOD-323_L1.7-W1.3-LS2.6-RD, F.Cu at (267.8, 73.7)
- J1: value Conn_01x02_Pin -> Mister
- J10: value Conn_01x02_Pin -> FoggerBasin
- J12: value Conn_01x03_Pin -> Moisture Sensor 3
- J13: value Conn_01x03_Pin -> Moisture Sensor 2
- J14: value Conn_01x03_Pin -> UART
- J15: value Conn_01x04_Pin -> FAE Fan
- J16: value Conn_01x02_Pin -> DrainLevel
- J2: value Conn_01x03_Pin -> Moisture Sensor 1
- J3: value Conn_01x04_Pin -> SCD30
- J4: value Conn_01x02_Pin -> Heater Fans
- J5: value Conn_01x02_Pin -> Fogger Solenoid
- J6: value Conn_01x02_Pin -> Drain Solenoid
- J7: value Conn_01x02_Pin -> Water Solenoid
- J8: value Conn_01x02_Pin -> Glycol Solenoid
- J9: value Conn_01x02_Pin -> CircFan
- LED1: renamed from LEDOn1; value EL304RD -> LED On
- LED10: renamed from Piezo1; value EL304RD -> Mister
- LED11: renamed from FAEFan1; value EL304RD -> FAE
- LED2: renamed from 12V_On1; value EL304RD -> 12V On
- LED3: renamed from CircFanLED1; value EL304RD -> CircFan
- LED4: renamed from GlycolSolenoidLED1; value EL304RD -> Glycol Solenoid
- LED5: renamed from WaterSolenoidLED1; value EL304RD -> Water Solenoid
- LED6: renamed from DrainSolenoidLED1; value EL304RD -> Drain Solenoid
- LED7: renamed from FoggerFillSolenoidLED1; value EL304RD -> Fogger Solenoid
- LED8: renamed from HeaterFansLED1; value EL304RD -> Heater Fans
- LED9: renamed from HeaterOnLED1; value EL304RD -> Heating Element
- P1: renamed from 12V_IN1; value Screw Terminal -> 12V_In
- moved SW4 104.5 mm to (202.4, 134.2)
- moved J10 75.1 mm to (217.5, 140.4), turned to 90 degrees
- moved LED10 58.5 mm to (274.9, 124.2)
- moved LED3 58.5 mm to (274.3, 112.7)
- moved LED7 58.5 mm to (274.8, 135.2)
- moved R33 58.5 mm to (278.8, 112.5)
- moved R39 58.5 mm to (279.1, 135.2)
- moved LED1 58.5 mm to (274.6, 140.2)
- moved LED11 58.5 mm to (274.6, 100.7)
- moved LED4 58.5 mm to (274.6, 117.2)
- moved LED5 58.5 mm to (274.1, 120.7)
- moved LED6 58.5 mm to (274.6, 130.2)
- moved LED9 58.5 mm to (274.6, 105.9)
- moved R35 58.5 mm to (278.8, 125.2)
- moved R36 58.5 mm to (279.9, 117.7)
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Connections:
- 12V_IN2 pad 1: Net-(12V_IN2-Pad1) -> 120V_IN
- 12V_IN2 pad 2: 120V_IN -> Net-(12V_IN2-Pad2)
- U10 pad 3: Net-(12V_IN2-Pad1) -> Net-(12V_IN2-Pad2)
- U10 pad 4: Net-(12V_IN2-Pad1) -> Net-(12V_IN2-Pad2)
Routing:
- net 120V_IN: track 44.4 -> 0.00 mm
- net ACS712_VOUT: track 1.84 -> 32.7 mm
- net Net-(K1-COIL1): track 30.9 -> 0.00 mm
- net Net-(K1-NO): track 26.2 -> 0.00 mm
- net Net-(12V_IN2-Pad1): track 8.29 -> 0.00 mm
- net KSD_Fault_RB: track 1.25 -> 6.97 mm
- net 5V_RB: track 5.24 -> 0.06 mm
- net Net-(U10-FILTER): track 2.24 -> 1.64 mm
- removed copper zone on F.Cu, net 12V_RB
- removed copper zone on B.Cu, net GND_RB
Other:
- board size 191.2 x 138.5 mm -> 190.3 x 138.6 mm

Commit message: pcb stuff
Parts:
- removed 12V_IN2: Screw Terminal, easyeda2kicad:CONN-TH_2P-P5.00_CPC3703CTR
- added CN1: KF237-5.08-1P, easyeda2kicad:CONN-TH_KF237-5.08-1P, F.Cu at (76.8, 174.9)
- added CN4: KF237-5.08-1P, easyeda2kicad:CONN-TH_KF237-5.08-1P, F.Cu at (77.0, 152.1)
- moved U10 50.2 mm to (70.9, 167.1), turned to 0 degrees
- moved C21 47.9 mm to (68.0, 164.0), turned to 90 degrees
- moved C22 43.6 mm to (72.3, 162.4), turned to 180 degrees
- moved R18 42.6 mm to (42.3, 157.6), turned to 180 degrees
- moved K1 42.2 mm to (57.7, 164.9), turned to -90 degrees
- moved R16 41.7 mm to (44.5, 151.2)
- moved U9 37.1 mm to (47.8, 160.7), turned to 90 degrees
- moved CN3 32.7 mm to (36.3, 164.1), turned to 90 degrees
- moved U3 2.98 mm to (53.9, 83.8)
Connections:
- net Net-(12V_IN2-Pad2) renamed 120V_Out
- net Net-(K1-NO) renamed NO_ACS
- CN3 pad 1: 12V_RB -> Net-(K1-COIL1)
- CN3 pad 2: Net-(K1-COIL1) -> 12V_RB
Routing:
- net Net-(K1-COIL1): track 0.00 -> 33.3 mm
- net ACS712_VOUT: track 32.7 -> 0.00 mm
- net NO_ACS: track 0.00 -> 20.6 mm
- net 12V_RB: track 0.00 -> 20.0 mm
- net 120V_IN: track 0.00 -> 18.6 mm
- net KSD_Fault_RB: track 6.97 -> 0.00 mm
- net 120V_Out: track 0.00 -> 6.83 mm
- net Net-(U10-FILTER): track 1.64 -> 0.00 mm
Other:
- board size 190.3 x 138.6 mm -> 190.3 x 147.1 mm
