File: GrowChamberPCB/GrowChamberPCB.kicad_pcb (KiCad board)
At the start: 2 copper layers, 190.3 x 105.6 mm, 154 parts, among them CN2 RelayBoard Interconnect, CN3 Connector_RB, J1 Mister, J10 FoggerBasin, J12 Moisture Sensor 3, J13 Moisture Sensor 2, J14 UART, J15 FAE Fan, J16 DrainLevel, J2 Moisture Sensor 1, J3 SCD30, J4 Heater Fans, J5 Fogger Solenoid, J6 Drain Solenoid, J7 Water Solenoid, J8 Glycol Solenoid, J9 CircFan, P1 12V_In, P2 12V_In, Q1 AO3400A_C347475, Q10 NPN, Q11 AO3400A_C347475, Q12 NPN, Q13 AO3400A_C347475, Q14 NPN, Q15 NPN, Q16 AO3400A_C347475, Q2 NPN, Q3 AO3400A_C347475, Q4 NPN, Q5 AO3400A_C347475, Q6 NPN, Q7 AO3400A_C347475, Q8 BRT30N70P3, Q9 NPN, SW1 Reset_Button_Internal, SW2 ResetButton_External, SW3 Bootmode_Internal, SW4 BootMode_External, U1 MP2393GTL-Z, U11 1N4007W, U12 1N4007W, U13 1N4007W, U14 1N4007W, U15 1N4007W, U16 1N4007W, U17 1N4007W, U19 To Faceplate, U2 MCP1826S-3302E/DB, U20 PCA9555APW,118, U3 ESP32-S3-WROOM-1U-N8R8, U4 To Faceplate, U5 1N4007W, U6 CR2013-MI2120, U7 TC4428EOA, U8 W25Q128JVSIQTR, U9 1N4007W

Commit message: forgot to save pcb
Parts:
- moved RLY1 11.4 mm to (54.2, 171.4)
- moved U9 11.4 mm to (42.0, 171.1)
- moved P2 11.4 mm to (61.7, 180.9)
Changed lines of the file:
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@@
 	(footprint "easyeda2kicad:RELAY-TH_G5NB-1A-E-DCXX"
 		(layer "F.Cu")
-		(at 65.43 173.24)
+		(at 54.18 171.43)
 		(property "Reference" "RLY1"
 			(at 0 -6.35 0)
@@
 	(footprint "easyeda2kicad:SOD-123FL_L2.7-W1.8-LS3.7-RD"
 		(layer "F.Cu")
-		(at 53.2 172.88 -90)
+		(at 41.95 171.07 -90)
 		(property "Reference" "U9"
 			(at 0 -4 90)
@@
 	(footprint "easyeda2kicad:CONN-TH_2P-P5.00_CPC3703CTR"
 		(layer "F.Cu")
-		(at 72.99 182.69 90)
+		(at 61.74 180.88 90)
 		(descr "WJ127-5.0-2P")
 		(property "Reference" "P2"

Commit message: Removed 3.3V, wired some stuff
Parts:
- removed 12V_IN4: Screw Terminal, easyeda2kicad:CONN-TH_2P-P5.00_CPC3703CTR
- removed C10, C11, C9: 4.7uF X7R, easyeda2kicad:C0603
- removed CN2: RelayBoard Interconnect, easyeda2kicad:CONN-TH_5P-P5.00_WJ127-5.0-5P
- removed CN3: Connector_RB, easyeda2kicad:CONN-TH_5P-P5.00_WJ127-5.0-5P
- removed R5: 7.68K, easyeda2kicad:R0603
- removed U16: 1N4007W, easyeda2kicad:SOD-123FL_L2.7-W1.8-LS3.7-RD
- removed U2: MCP1826S-3302E/DB, easyeda2kicad:SOT-223-3_L6.7-W3.7-P2.30-LS7.0-BR
- added C21: 10uF, easyeda2kicad:C0603, F.Cu at (77.8, 165.9)
- added L3: ZHT103, easyeda2kicad:IND-TH_L18.2-W10.2-P12.00-D0.9_ZHT103, F.Cu at (69.8, 161.0)
- added R16: 50, easyeda2kicad:R0603, F.Cu at (78.0, 162.9)
- added R18: 100k, easyeda2kicad:R0603, F.Cu at (76.3, 163.0)
- added R45: 100k, easyeda2kicad:R0603, F.Cu at (76.3, 165.9)
- added R46: 100K, easyeda2kicad:R0603, F.Cu at (60.4, 119.8)
- added R47: 100K, easyeda2kicad:R0603, F.Cu at (62.4, 124.0)
- added R48: 10K, easyeda2kicad:R0603, F.Cu at (62.5, 125.6)
- added R49: 10K, easyeda2kicad:R0603, F.Cu at (60.4, 118.2)
- added R50: 20K, easyeda2kicad:R0603, F.Cu at (60.6, 95.2)
- added U10: 1N4007W, easyeda2kicad:SOD-123FL_L2.7-W1.8-LS3.7-RD, F.Cu at (72.0, 49.4)
- P2: value 12V_In -> 120V
- R3: value 15K -> 13K
- R35, R43: value 270 -> 1k
- moved Power_FP1 194.1 mm to (246.8, 69.9)
- moved J14 169.1 mm to (255.0, 70.3)
- moved U15 155.5 mm to (32.0, 49.9), turned to 90 degrees
- moved Q7 151.8 mm to (53.7, 45.5)
- moved U12 147.0 mm to (52.2, 49.6), turned to 90 degrees
- moved Q6 146.4 mm to (57.7, 45.5)
- moved R24 144.1 mm to (55.2, 49.2), turned to -90 degrees
- moved C19 141.5 mm to (-16.2, 55.0)
- moved C18 141.3 mm to (-16.1, 52.6)
- moved R23 140.2 mm to (58.3, 49.2), turned to 90 degrees
- moved Q5 139.1 mm to (73.5, 45.3)
- moved L1 137.9 mm to (44.4, 81.0)
- moved Q16 134.7 mm to (34.0, 45.9)
- moved Q4 133.4 mm to (77.5, 45.3)
- moved R22 130.9 mm to (75.0, 49.0), turned to -90 degrees
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Connections:
- D1 pad 5: 5V -> VBUS
- D4 pad 2: GND_FP -> GND
- P2 pad 1: 120V_To_ACS -> 120V_Out
- P2 pad 2: 120V_Out -> 120V_IN
- R17 pad 1: Net-(Q1-G) -> 12V
- R17 pad 2: 12V -> Net-(Q1-G)
- R20 pad 1: Net-(Q2-C) -> 12V
- R20 pad 2: 12V -> Net-(Q2-C)
- R22 pad 1: Net-(Q4-C) -> 12V
- R22 pad 2: 12V -> Net-(Q4-C)
- R24 pad 1: Net-(Q6-C) -> 12V
- R24 pad 2: 12V -> Net-(Q6-C)
- R26 pad 1: Net-(Q10-C) -> 12V
- R26 pad 2: 12V -> Net-(Q10-C)
- R28 pad 1: Net-(Q12-C) -> 12V
- R28 pad 2: 12V -> Net-(Q12-C)
- R3 pad 1: FB -> GND
- R31 pad 1: Net-(Q14-C) -> 12V
- R31 pad 2: 12V -> Net-(Q14-C)
- R35 pad 2: 5V_FP -> 12V_FP
- R43 pad 2: 5V_FP -> 12V_FP
- RLY1 pad 1: 12V_RB -> Heater_ON
- RLY1 pad 2: unconnected-(RLY1-Pad2) -> 120V_Out
- RLY1 pad 3: 120V_Out -> 120V_IN
- RLY1 pad 4: Net-(U9-K) -> 12V
- U12 pad 2: DrainSol -> WaterSol
- U13 pad 2: WaterSol -> GlycolSol
- U14 pad 2: GlycolSol -> Circ_Fan
- U15 pad 2: Circ_Fan -> Heater_ON
- U3 pad 12: Fogger_Basin_Float_Switch -> Net-(U3-IO8)
- U3 pad 7: Drain_Level -> Net-(U3-IO7)
- U7 pad 5: Piezo2 -> Piezo1
- U7 pad 7: Piezo1 -> Piezo2
- U9 pad 1: Net-(U9-K) -> 12V
- U9 pad 2: 12V_RB -> Heater_ON
- USB1 pad A4B9: 5V -> VBUS
- USB1 pad B4A9: 5V -> VBUS
Routing:
- net Net-(C21-Pad2): track 0.00 -> 13.6 mm
- net VBUS: track 0.00 -> 12.5 mm, vias 0 -> 2
- net D+: track 0.00 -> 11.7 mm
- net D-: track 0.00 -> 11.7 mm
- net LEDs: track 0.00 -> 11.3 mm
- net KSD_Fault: track 0.00 -> 11.1 mm
- net Heater_ON: track 0.00 -> 5.92 mm
- net Net-(Q8-G): track 0.00 -> 5.54 mm
- net Net-(Q14-C): track 0.00 -> 4.46 mm
- net DC_Display: track 0.00 -> 4.07 mm
- net Net-(USB1-CC1): track 0.00 -> 3.28 mm
- net Net-(USB1-CC2): track 0.00 -> 2.75 mm
- net Net-(Q14-B): track 0.00 -> 2.18 mm
- net Net-(U8-IO3): track 0.00 -> 2.18 mm
- net Net-(U8-IO2): track 0.00 -> 2.15 mm
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- added copper zone on F.Cu, net 120V_IN
- added copper zone on F.Cu, net 120V_Out
- added copper zone on F.Cu, net 12V
- added copper zone on B.Cu, net GND
Other:
- board size 190.3 x 105.6 mm -> 192 x 102.2 mm

Commit message: failing to route the board
Parts:
- removed D1: SRV05-4_C2836319, easyeda2kicad:SOT-23-6_L2.9-W1.6-P0.95-LS2.8-BL
- removed LED_To_Connector1: Screw Terminal, easyeda2kicad:CONN-TH_2P-P5.00_CPC3703CTR
- removed Q14: NPN, easyeda2kicad:SOT-23-3_L3.0-W1.7-P0.95-LS2.9-BR
- removed Q16: AO3400A_C347475, easyeda2kicad:SOT-23-3_L2.9-W1.3-P1.90-LS2.4-BR
- removed R43: 1k, easyeda2kicad:R0603
- removed U11, U15: 1N4007W, easyeda2kicad:SOD-123FL_L2.7-W1.8-LS3.7-RD
- removed U19, U4: To Faceplate, easyeda2kicad:IDC-TH_26P-P2.54_ZX-IDC2.54-2-13PZZ
- added D19: USBLC6-2SC6, easyeda2kicad:SOT-23-6_L2.9-W1.6-P0.95-LS2.8-BL, F.Cu at (-6.50, 82.2)
- added J11: TP, TestPoint:TestPoint_Pad_D2.0mm, F.Cu at (58.0, 22.2)
- added J17: TP, TestPoint:TestPoint_Pad_D2.0mm, F.Cu at (64.0, 27.2)
- added J18: TP, TestPoint:TestPoint_Pad_D2.0mm, F.Cu at (57.5, 14.0)
- added J19: TP, TestPoint:TestPoint_Pad_D2.0mm, F.Cu at (46.0, 21.8)
- added J20: TP, TestPoint:TestPoint_Pad_D2.0mm, F.Cu at (40.5, 26.8)
- added J21: TP, TestPoint:TestPoint_Pad_D2.0mm, F.Cu at (49.8, 21.8)
- added J22: TP, TestPoint:TestPoint_Pad_D2.0mm, F.Cu at (-19.0, 32.0)
- added J23: TP, TestPoint:TestPoint_Pad_D2.0mm, F.Cu at (-33.5, 24.8)
- added J24: TP, TestPoint:TestPoint_Pad_D2.0mm, F.Cu at (-24.2, 15.0)
- added J25: TP, TestPoint:TestPoint_Pad_D2.0mm, F.Cu at (-33.6, 51.1)
- added J26: TP, TestPoint:TestPoint_Pad_D2.0mm, F.Cu at (-47.0, 42.5)
- added J27: TP, TestPoint:TestPoint_Pad_D2.0mm, F.Cu at (-6.75, 43.5)
- added J28: TP, TestPoint:TestPoint_Pad_D2.0mm, F.Cu at (-15.2, 32.0)
- added J29: TP, TestPoint:TestPoint_Pad_D2.0mm, F.Cu at (-37.2, 24.8)
- added J30: TP, TestPoint:TestPoint_Pad_D2.0mm, F.Cu at (-20.5, 15.0)
- added J31: TP, TestPoint:TestPoint_Pad_D2.0mm, F.Cu at (-37.4, 51.1)
- added J32: TP, TestPoint:TestPoint_Pad_D2.0mm, F.Cu at (-43.2, 42.5)
- added J33: TP, TestPoint:TestPoint_Pad_D2.0mm, F.Cu at (-10.5, 43.5)
- added J34: TP, TestPoint:TestPoint_Pad_D2.0mm, F.Cu at (-5.00, 27.5)
- added J35: TP, TestPoint:TestPoint_Pad_D2.0mm, F.Cu at (-47.5, 29.2)
- added J36: TP, TestPoint:TestPoint_Pad_D2.0mm, F.Cu at (-10.2, 10.5)
- added J37: TP, TestPoint:TestPoint_Pad_D2.0mm, F.Cu at (-47.6, 55.6)
- added J38: TP, TestPoint:TestPoint_Pad_D2.0mm, F.Cu at (-33.0, 38.0)
- added J39: TP, TestPoint:TestPoint_Pad_D2.0mm, F.Cu at (-20.8, 48.0)
- added J40: TP, TestPoint:TestPoint_Pad_D2.0mm, F.Cu at (83.5, 49.8)
- added J41: TP, TestPoint:TestPoint_Pad_D2.0mm, F.Cu at (71.2, 49.8)
- added J42: TP, TestPoint:TestPoint_Pad_D2.0mm, F.Cu at (20.8, 134.0)
- added J43: TP, TestPoint:TestPoint_Pad_D2.0mm, F.Cu at (40.0, 132.5)
- added J44: TP, TestPoint:TestPoint_Pad_D2.0mm, F.Cu at (-62.3, 73.8)
- added J45: TP, TestPoint:TestPoint_Pad_D2.0mm, F.Cu at (-69.8, 73.8)
- added J46: TP, TestPoint:TestPoint_Pad_D2.0mm, F.Cu at (-73.0, 129.0)
- added J47: TP, TestPoint:TestPoint_Pad_D2.0mm, F.Cu at (21.0, 25.0)
- added J48: TP, TestPoint:TestPoint_THTPad_2.0x2.0mm_Drill1.0mm, F.Cu at (16.0, 25.0)
- added J49: TP, TestPoint:TestPoint_Pad_D2.0mm, F.Cu at (149.5, 19.0)
- added J50: TP, TestPoint:TestPoint_THTPad_2.0x2.0mm_Drill1.0mm, F.Cu at (144.5, 19.5)
- added J51: Conn_01x12, Connector_PinSocket_2.54mm:PinSocket_1x12_P2.54mm_Vertical, F.Cu at (153.7, 68.3)
- added J52: Conn_01x12, Connector_PinSocket_2.54mm:PinSocket_1x12_P2.54mm_Vertical, F.Cu at (158.2, 68.3)
- added J53: Conn_01x12, Connector_PinSocket_2.54mm:PinSocket_1x12_P2.54mm_Vertical, F.Cu at (107.0, 73.3)
- added J54: Conn_01x12, Connector_PinSocket_2.54mm:PinSocket_1x12_P2.54mm_Vertical, F.Cu at (108.0, 57.8)
- added LED12: LED On, easyeda2kicad:LED-TH_BD3.9-P2.54-RD_RED, F.Cu at (193.8, 76.5)
- added P3: Screw Terminal, easyeda2kicad:CONN-TH_2P-P5.00_CPC3703CTR, F.Cu at (30.5, 18.5)
- added Q17: NPN, easyeda2kicad:SOT-23-3_L3.0-W1.7-P0.95-LS2.9-BR, F.Cu at (62.0, 16.0)
- added Q18: MOSFET, easyeda2kicad:SOT-23-3_L2.9-W1.3-P1.90-LS2.4-BR, F.Cu at (62.5, 19.8)
- added R5: 33, easyeda2kicad:R0603, F.Cu at (-3.25, 114.2)
- added R51: 1k, easyeda2kicad:R0603, F.Cu at (-19.0, 70.5)
- added R52: 1k, easyeda2kicad:R0603, F.Cu at (62.0, 13.0)
- added R53: 1M, easyeda2kicad:R0603, F.Cu at (57.2, 18.8)
- Q1, Q11, Q13, Q3, Q5, Q7: value AO3400A_C347475 -> MOSFET
- R29, R35: value 1k -> 75
- R31: value 1M -> 75
- R34: value 1k -> 1M
- U8: value W25Q128JVSIQTR -> Memory
- moved J6 168.6 mm to (128.0, 27.0)
- moved J7 168.3 mm to (127.7, 35.5)
- moved J8 161.7 mm to (134.5, 43.5)
- moved C2 159.7 mm to (-82.0, 118.0)
- moved C1 159.5 mm to (-82.0, 114.7)
- moved C6 147.6 mm to (-82.0, 124.7), turned to 0 degrees
- moved C4 146.7 mm to (-76.8, 117.0)
- moved R15 146.5 mm to (-25.5, 116.8), turned to 0 degrees
- moved U1 146.5 mm to (-81.2, 109.6), turned to 0 degrees
- moved C3 146.4 mm to (-76.8, 114.3), turned to 0 degrees
- moved C7 145.2 mm to (-76.8, 119.7), turned to 0 degrees
- moved R3 144.3 mm to (-71.8, 119.0), turned to 0 degrees
- moved R4 143.7 mm to (-71.8, 121.5)
- moved R2 143.5 mm to (-71.8, 116.5), turned to 0 degrees
- moved C5 142.8 mm to (-82.0, 121.3), turned to 0 degrees
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Connections:
- net Net-(U3-IO7) renamed GPIO7
- net Net-(U3-IO8) renamed GPIO8
- C16 pad 1: D+ -> Out_D+
- C17 pad 1: D- -> Out_D-
- C5 pad 1: 5V -> 3.3V
- C6 pad 1: 5V -> 3.3V
- C8 pad 1: 5V -> 3.3V
- D13 pad 1: GPIO1_FP -> GPIO4_FP
- D13 pad 3: GPIO2_FP -> /Faceplate/3.3V ESD/IO2
- D13 pad 4: Drain_Level_FP -> GPIO1_FP
- D13 pad 6: GPIO4_FP -> GPIO2_FP
- D16 pad 1: /Faceplate/Data Line ESD/IO1 -> EN_FP
- D16 pad 3: EN_FP -> BootMode_FP
- D16 pad 4: Fogger_Basin_Float_Switch_FP -> Drain_Level_FP
- D16 pad 6: BootMode_FP -> Fogger_Basin_Float_Switch_FP
- D18 pad 1: Display_Reset -> unconnected-(D18-Pad1)
- D18 pad 3: unconnected-(D18-Pad3) -> CS_SD
- D18 pad 4: unconnected-(D18-Pad4) -> MOSI
- D18 pad 6: unconnected-(D18-Pad6) -> MISO
- D2 pad 1: EN -> BootMode
- D2 pad 3: BootMode -> EN
- D2 pad 4: CS_SD -> SCK
- D2 pad 6: MOSI -> unconnected-(D2-Pad6)
- D3 pad 3: DC_Display -> Display_Reset
- D3 pad 4: MISO -> DC_Display
- D3 pad 6: SCK -> MOSI
- L1 pad 2: 5V -> 3.3V
- R18 pad 1: 5V -> 3.3V
- R29 pad 1: Heater_Switch -> Net-(LED10-A)
- R29 pad 2: Net-(Q14-B) -> 3.3V_FP
- R31 pad 1: 12V -> Net-(LED12-A)
- R31 pad 2: Net-(Q14-C) -> 3.3V_FP
- R35 pad 1: Net-(LED10-A) -> Net-(LED11-A)
- R35 pad 2: 12V_FP -> 3.3V_FP
- R4 pad 2: 5V -> 3.3V
- R6 pad 2: BootMode -> Net-(R6-Pad2)
- R8 pad 1: D- -> Out_D-
- R9 pad 1: D+ -> Out_D+
- SW3 pad 1: unconnected-(SW3-Pad1) -> Net-(R6-Pad2)
- U20 pad 24: 5V_FP -> unconnected-(U20-VDD-Pad24)
- U20 pad 9: unconnected-(U20-P0_5-Pad9) -> Net-(LED12-K)
- U3 pad 18: External_Fan_PWM -> Net-(U3-IO10)
- U3 pad 23: CS_SD -> unconnected-(U3-IO21-Pad23)
- U3 pad 24: Display_Reset -> unconnected-(U3-IO47-Pad24)
- U3 pad 25: CS_Memory -> unconnected-(U3-IO48-Pad25)
- U3 pad 26: Fan_Tach -> CS_Display
- U3 pad 31: CS_Display -> Display_Reset
- U3 pad 33: SCK -> CS_Memory
- U3 pad 34: MOSI -> CS_SD
- U3 pad 35: MISO -> MOSI
- U3 pad 38: GPIO2 -> MISO
- U3 pad 39: GPIO1 -> Net-(U3-IO1)
- U3 pad 4: GPIO4 -> unconnected-(U3-IO4-Pad4)
Routing:
- net GND: track 0.00 -> 36.5 mm, vias 0 -> 12
- net Net-(J32-Pin_1): track 0.00 -> 9.36 mm
- net Net-(J31-Pin_1): track 0.00 -> 9.36 mm
- net Net-(J11-Pin_1): track 0.00 -> 8.93 mm
- net D-: track 11.7 -> 4.20 mm
- net Net-(J41-Pin_1): track 13.6 -> 20.5 mm
- net 120V_IN: track 0.00 -> 6.67 mm
- net D+: track 11.7 -> 5.32 mm
- net LEDs: track 11.3 -> 17.7 mm
- net 120V_Out: track 0.52 -> 6.46 mm
- net WaterSol: track 0.00 -> 5.22 mm
- net GlycolSol: track 0.00 -> 5.22 mm
- net GPIO18: track 0.00 -> 5.10 mm
- net 12V: track 1.51 -> 6.50 mm
- net Net-(J19-Pin_1): track 5.54 -> 10.2 mm
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- removed copper zone on F.Cu, net 120V_IN
- removed copper zone on F.Cu, net 120V_Out
- removed copper zone on F.Cu, net 12V
- removed copper zone on B.Cu, net GND
Other:
- board size 192 x 102.2 mm -> 100 x 100 mm
- board text added: "120V Keepout"

Commit message: almost done routing
Parts:
- removed D2: SRV05-4_C2836319, easyeda2kicad:SOT-23-6_L2.9-W1.6-P0.95-LS2.8-BL
- removed J51, J52, J53, J54: Conn_01x12, Connector_PinSocket_2.54mm:PinSocket_1x12_P2.54mm_Vertical
- added D1: SRV05-4_C2836319, easyeda2kicad:SOT-23-6_L2.9-W1.6-P0.95-LS2.8-BL, F.Cu at (77.0, 102.5)
- added R43: 33, easyeda2kicad:R0603, F.Cu at (35.5, 101.0)
- added R54: 33, easyeda2kicad:R0603, F.Cu at (35.5, 99.5)
- added R55: 33, easyeda2kicad:R0603, F.Cu at (36.2, 96.4)
- added R56: 33, easyeda2kicad:R0603, F.Cu at (35.5, 102.8)
- added R57: 33, easyeda2kicad:R0603, F.Cu at (37.4, 93.2)
- added U2: ZX-IDC2.54-2-13PZZ, easyeda2kicad:IDC-TH_26P-P2.54_ZX-IDC2.54-2-13PZZ, F.Cu at (210.5, 38.9)
- added U4: ZX-IDC2.54-2-13PZZ, easyeda2kicad:IDC-TH_26P-P2.54_ZX-IDC2.54-2-13PZZ, F.Cu at (76.7, 77.6)
- moved C1 256.3 mm to (174.3, 113.2)
- moved C2 256.3 mm to (174.3, 116.5)
- moved C5 256.3 mm to (174.3, 119.8)
- moved C6 256.3 mm to (174.3, 123.2)
- moved J46 256.3 mm to (183.3, 127.5)
- moved L1 256.3 mm to (174.3, 130.0)
- moved R1 256.3 mm to (184.6, 112.6)
- moved R2 256.3 mm to (184.6, 115.0)
- moved R3 256.3 mm to (184.6, 117.5)
- moved R4 256.3 mm to (184.6, 120.0)
- moved R50 256.3 mm to (184.6, 122.5)
- moved U1 256.3 mm to (175.1, 108.2)
- moved C3 256.3 mm to (179.4, 112.8)
- moved C4 256.3 mm to (179.4, 115.5)
- moved C7 256.3 mm to (179.4, 118.2)
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Connections:
- D18 pad 1: unconnected-(D18-Pad1) -> CS_SD
- D18 pad 3: CS_SD -> SCK
- D18 pad 4: MOSI -> MISO
- D18 pad 6: MISO -> MOSI
- D3 pad 1: CS_Display -> Display_Reset
- D3 pad 3: Display_Reset -> CS_Display
- D3 pad 4: DC_Display -> MOSI
- D3 pad 6: MOSI -> DC_Display
- J21 pad 1: GPIO18 -> LEDIO
- J34 pad 1: GPIO13 -> HeaterFans_IO
- J35 pad 1: GPIO14 -> FoggerSol_IO
- J36 pad 1: GPIO15 -> DrainSolIO
- J37 pad 1: GPIO16 -> WaterSol_IO
- J38 pad 1: GPIO17 -> GlycolSol_IO
- J39 pad 1: GPIO46 -> CircFan_IO
- R19 pad 1: GPIO14 -> FoggerSol_IO
- R21 pad 1: GPIO15 -> DrainSolIO
- R23 pad 1: GPIO16 -> WaterSol_IO
- R25 pad 1: GPIO17 -> GlycolSol_IO
- R27 pad 1: GPIO46 -> CircFan_IO
- R30 pad 1: GPIO13 -> HeaterFans_IO
- R32 pad 1: GPIO18 -> LEDIO
- R46 pad 1: GPIO7 -> DrainLevel_IO
- R47 pad 1: GPIO8 -> FloatSwitch_IO
- R48 pad 1: GPIO8 -> FloatSwitch_IO
- R49 pad 1: GPIO7 -> DrainLevel_IO
- R5 pad 1: Net-(U3-IO1) -> Net-(U3-IO8)
- R51 pad 2: Net-(U3-IO10) -> Net-(U3-IO2)
- U3 pad 10: GPIO17 -> Net-(U3-IO17)
- U3 pad 11: GPIO18 -> Net-(U3-IO18)
- U3 pad 12: GPIO8 -> Net-(U3-IO8)
- U3 pad 16: GPIO46 -> WaterSol_IO
- U3 pad 17: KSD_Fault -> GlycolSol_IO
- U3 pad 18: Net-(U3-IO10) -> CircFan_IO
- U3 pad 19: Fogger_PWM -> FoggerSol_IO
- U3 pad 20: Heater_Switch -> HeaterFans_IO
- U3 pad 21: GPIO13 -> LEDIO
- U3 pad 22: GPIO14 -> Heater_Switch
- U3 pad 23: unconnected-(U3-IO21-Pad23) -> Fogger_PWM
- U3 pad 24: unconnected-(U3-IO47-Pad24) -> KSD_Fault
- U3 pad 25: unconnected-(U3-IO48-Pad25) -> SDA
- U3 pad 26: CS_Display -> SCL
- U3 pad 31: Display_Reset -> Soil_Moisture4
- U3 pad 32: DC_Display -> Soil_Moisture2
- U3 pad 33: CS_Memory -> Soil_Moisture1
- U3 pad 34: CS_SD -> DrainLevel_IO
- U3 pad 35: MOSI -> FloatSwitch_IO
- U3 pad 38: MISO -> Net-(U3-IO2)
- U3 pad 39: Net-(U3-IO1) -> Fan_Tach
- U3 pad 4: unconnected-(U3-IO4-Pad4) -> DrainSolIO
- U3 pad 5: SDA -> Net-(U3-IO5)
- U3 pad 6: SCL -> Display_Reset
- U3 pad 7: GPIO7 -> Net-(U3-IO7)
- U3 pad 8: GPIO15 -> DC_Display
- U3 pad 9: GPIO16 -> Net-(U3-IO16)
Routing:
- net Heater_Switch: track 4.16 -> 101.8 mm
- net LEDIO: track 0.00 -> 96.4 mm
- net WaterSol_IO: track 0.00 -> 85.1 mm
- net GlycolSol_IO: track 0.00 -> 79.9 mm
- net FoggerSol_IO: track 0.00 -> 76.9 mm
- net HeaterFans_IO: track 0.00 -> 73.6 mm
- net Fogger_PWM: track 0.00 -> 72.4 mm
- net KSD_Fault: track 13.1 -> 82.0 mm, vias 0 -> 2
- net CS_SD: track 0.00 -> 67.0 mm
- net SCK: track 0.55 -> 65.5 mm
- net EN: track 0.00 -> 64.5 mm, vias 0 -> 2
- net CircFan_IO: track 0.00 -> 62.0 mm
- net MOSI: track 0.00 -> 57.6 mm
- net Soil_Moisture4: track 0.00 -> 54.7 mm, vias 0 -> 1
- net MISO: track 0.64 -> 52.3 mm
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- added copper zone on B.Cu, net GND

Commit message: working on pcb
Parts:
- removed C1, C2: 22uF X7R, easyeda2kicad:C1206
- removed C3: 1nF, easyeda2kicad:C0603
- removed C4: 1uF, easyeda2kicad:C0603
- removed C7: 6.8nF, easyeda2kicad:C0603
- removed C8: 10pF, easyeda2kicad:C0603
- removed J46: TP, TestPoint:TestPoint_Pad_D2.0mm
- removed R1: 20, easyeda2kicad:R0603
- removed R14: 10K, easyeda2kicad:R0603
- removed R2: 604K, easyeda2kicad:R0603
- removed R3: 13K, easyeda2kicad:R0603
- removed R4: 40.2K, easyeda2kicad:R0603
- removed U1: MP2393GTL-Z, easyeda2kicad:SOT-583-8_L2.1-W1.2-P0.50-LS1.6-BL
- removed U6: CR2013-MI2120, Connector_PinHeader_2.54mm:PinHeader_1x14_P2.54mm_Vertical
- added C22: 10uF, easyeda2kicad:C0603, F.Cu at (50.2, 45.2)
- added C23: 100nF, easyeda2kicad:C0603, F.Cu at (49.2, 51.0)
- added J51: TP, TestPoint:TestPoint_Pad_D2.0mm, F.Cu at (16.0, 25.0)
- added J52: TP, TestPoint:TestPoint_Pad_D2.0mm, F.Cu at (44.8, 62.0)
- added J53: TP, TestPoint:TestPoint_Pad_D2.0mm, F.Cu at (21.0, 24.8)
- added LED13: 12V On, easyeda2kicad:LED-TH_BD3.9-P2.54-RD_RED, F.Cu at (-3.47, 37.8)
- added R58: 33, easyeda2kicad:R0603, F.Cu at (68.5, 93.5)
- added R59: 33, easyeda2kicad:R0603, F.Cu at (65.2, 92.2)
- added R60: 1k, easyeda2kicad:R0603, F.Cu at (-4.08, 41.6)
- added U11: AP63203WU-7, easyeda2kicad:TSOT-26_L2.9-W1.6-P0.95-LS2.8-BL, F.Cu at (51.0, 48.2)
- J47: value TP -> Conn_01x04; footprint TestPoint:TestPoint_Pad_D2.0mm -> Connector_PinSocket_2.54mm:PinSocket_1x04_P2.54mm_Vertical
- J48: value TP -> Conn_01x09; footprint TestPoint:TestPoint_THTPad_2.0x2.0mm_Drill1.0mm -> Connector_PinSocket_2.54mm:PinSocket_1x09_P2.54mm_Vertical
- L1: value PRS8040-3R6MT -> ANR4030T3R9M; footprint easyeda2kicad:IND-SMD_L8.0-W8.0 -> easyeda2kicad:IND-SMD_L4.0-W4.0
- R50: value 20K -> 10K
- moved R50 158.9 mm to (29.1, 89.4), turned to 90 degrees
- moved L1 152.5 mm to (44.5, 50.0), turned to -90 degrees
- moved C6 147.0 mm to (43.8, 55.5), turned to -90 degrees
- moved C5 143.1 mm to (46.5, 55.5), turned to -90 degrees
- moved J47 53.2 mm to (18.5, 78.1)
- moved J48 44.9 mm to (23.3, 69.3)
- moved R10 25.3 mm to (56.0, 85.8), turned to 90 degrees
- moved R11 25.0 mm to (63.5, 86.8), turned to 90 degrees
- moved R15 15.9 mm to (27.9, 75.7), turned to -90 degrees
- moved C20 12.3 mm to (31.1, 89.4), turned to -90 degrees
- moved D18 11.4 mm to (18.5, 90.1), turned to 90 degrees
- moved D3 8.05 mm to (18.5, 73.0)
- moved J37 7.36 mm to (18.2, 45.8)
- moved R55 5.40 mm to (35.5, 101.8)
- moved R54 4.70 mm to (35.5, 94.8)
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Connections:
- D18 pad 1: CS_SD -> MOSI
- D18 pad 6: MOSI -> CS_SD
- D3 pad 4: MOSI -> unconnected-(D3-Pad4)
- J47 pad 1: 12V -> CS_SD
- J48 pad 1: GND -> 3.3V
- R43 pad 1: Net-(U3-IO17) -> Net-(U3-IO16)
- R5 pad 1: Net-(U3-IO8) -> Net-(U3-IO18)
- R50 pad 1: FB -> 3.3V
- R50 pad 2: Net-(C8-Pad2) -> Net-(U8-IO3)
- R54 pad 1: Net-(U3-IO16) -> Net-(U3-IO15)
- R54 pad 2: MOSI -> CS_Memory
- R55 pad 1: Net-(U3-IO7) -> Net-(U3-IO8)
- R56 pad 1: Net-(U3-IO18) -> Net-(U3-IO17)
- R56 pad 2: CS_Memory -> MOSI
- U20 pad 24: unconnected-(U20-VDD-Pad24) -> 3.3V_FP
- U3 pad 36: RXD0 -> Net-(U3-RXD0)
- U3 pad 37: TXD0 -> Net-(U3-TXD0)
- U3 pad 7: Net-(U3-IO7) -> DC_Display
- U3 pad 8: DC_Display -> Net-(U3-IO15)
- U4 pad 11: unconnected-(U4-Pad11) -> GlycolSol
- U4 pad 13: unconnected-(U4-Pad13) -> FoggerSol
- U4 pad 15: unconnected-(U4-Pad15) -> Heater Fans
- U4 pad 17: unconnected-(U4-Pad17) -> DrainSol
- U4 pad 19: unconnected-(U4-Pad19) -> Circ_Fan
- U4 pad 2: unconnected-(U4-Pad2) -> 3.3V
- U4 pad 4: unconnected-(U4-Pad4) -> 3.3V
- U4 pad 5: unconnected-(U4-Pad5) -> Heater_ON
- U4 pad 6: unconnected-(U4-Pad6) -> EN
- U4 pad 7: unconnected-(U4-Pad7) -> LEDs
- U4 pad 8: unconnected-(U4-Pad8) -> BootMode
- U4 pad 9: unconnected-(U4-Pad9) -> WaterSol
Routing:
- net WaterSol: track 5.22 -> 95.0 mm, vias 0 -> 1
- net GlycolSol: track 5.22 -> 90.1 mm, vias 0 -> 1
- net FoggerSol: track 5.22 -> 80.8 mm, vias 0 -> 1
- net Heater Fans: track 5.22 -> 73.2 mm, vias 0 -> 1
- net Heater_ON: track 9.95 -> 77.0 mm, vias 0 -> 3
- net Circ_Fan: track 5.22 -> 70.6 mm, vias 0 -> 3
- net LEDs: track 17.7 -> 81.3 mm, vias 0 -> 1
- net DrainSol: track 5.22 -> 50.9 mm, vias 0 -> 3
- net BootMode: track 19.5 -> 63.0 mm
- net GND: track 36.5 -> 79.5 mm, vias 12 -> 42
- net EN: track 64.5 -> 106.6 mm
- net CS_SD: track 67.0 -> 39.2 mm
- net SCK: track 65.5 -> 38.1 mm
- net RXD0: track 31.9 -> 21.9 mm
- net MOSI: track 57.6 -> 47.6 mm
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- added copper zone on F.Cu, net 12V
- added copper zone on F.Cu, net 3.3V
Other:
- outline, holes or cut-outs redrawn
