File: GrowChamberPCB/GrowChamberPCB.kicad_pcb (KiCad board)
At the start: 4 copper layers, 100 x 100 mm, 191 parts, among them J1 Mister, J10 FoggerBasin, J12 Moisture Sensor 3, J13 Moisture Sensor 2, J14 UART, J15 FAE Fan, J16 DrainLevel, J2 Moisture Sensor 1, J3 SCD30, J34 TP, J35 TP, J36 TP, J37 TP, J38 TP, J39 TP, J4 Heater Fans, J40 TP, J41 TP, J42 TP, J43 TP, J44 TP, J45 TP, J46 TP, J47 Conn_01x04, J48 Conn_01x09, J49 12V, J5 Fogger Solenoid, J50 Gnd, J51 TP, J52 TP, J53 TP, J54 TP, J55 TP, J56 TP, J57 TP, J58 TP, J59 TP, J6 Drain Solenoid, J60 TP, J7 Water Solenoid, J8 Glycol Solenoid, J9 CircFan, P1 12V_In, P2 120V, P3 LED Connector, Q10 AO3400A, Q11 AO3400A, Q12 AO3400A, Q13 AO3400A, Q14 AO3400A, Q15 AO3400A, Q16 AO3400A, Q7 AO3400A, SW1 TS-1088-AR02016, SW3 Bootmode_Internal, SW4 BootMode_External, SW5 On/Off, U11 SRV05-4A, U12 SRV05-4A, U13 SRV05-4A, U14 SRV05-4A, U15 SRV05-4A, U16 SRV05-4A, U17 SRV05-4A, U18 SRV05-4A, U2 2x13, U3 ESP32-S3-WROOM-1U-N8R8, U4 ZX-IDC2.54-2-13PZZ, U6 TPS5430DDAR, U7 TC4428EOA, U8 Memory

Commit message: fixing stuff
Parts:
- moved D1 0.79 mm to (147.0, 132.0)
- moved D3 0.73 mm to (147.0, 127.1)
- moved J15 0.73 mm to (142.2, 124.0)
- moved D7 0.72 mm to (141.6, 47.1)
- moved J1 0.65 mm to (142.0, 41.2)
- moved R39 0.60 mm to (164.4, 38.0)
- moved C20 0.57 mm to (80.7, 95.8)
- moved D2 0.56 mm to (100.3, 78.9)
- moved D6 0.52 mm to (141.6, 37.9)
- moved R16 0.40 mm to (160.3, 37.8)
Connections:
- U11 pad 2: GND_FP -> 3.3V_FP
- U11 pad 5: 3.3V_FP -> GND_FP
- U12 pad 2: GND_FP -> 3.3V_FP
- U12 pad 5: 3.3V_FP -> GND_FP
- U13 pad 2: GND_FP -> 3.3V_FP
- U13 pad 5: 3.3V_FP -> GND_FP
- U14 pad 2: GND_FP -> 3.3V
- U14 pad 5: 3.3V_FP -> GND
- U15 pad 2: GND_FP -> 3.3V_FP
- U15 pad 5: 3.3V_FP -> GND_FP
- U16 pad 2: GND_FP -> 3.3V
- U16 pad 5: 3.3V_FP -> GND
- U17 pad 2: GND_FP -> 3.3V
- U17 pad 5: 3.3V_FP -> GND
- U18 pad 2: GND_FP -> 3.3V
- U18 pad 5: 3.3V_FP -> GND
Routing:
- net 12V_FP: track 0.00 -> 71.7 mm, vias 0 -> 1
- net GND_FP: track 0.00 -> 8.60 mm, vias 0 -> 8
- net VBUS: track 8.31 -> 0.28 mm
- net SoilMoisture2_FP: track 32.5 -> 36.7 mm
- net 3.3V: track 0.00 -> 3.88 mm, vias 0 -> 3
- net MISO: track 36.9 -> 39.8 mm
- net Heater_ON: track 78.8 -> 76.5 mm, vias 1 -> 0
- net SCK: track 51.2 -> 49.3 mm
- net Net-(D2-K): track 13.3 -> 11.8 mm
- net External_Fan_PWM_FP: track 61.6 -> 60.3 mm
- net GND: track 0.00 -> 1.19 mm, vias 9 -> 10
- net D+: track 27.4 -> 26.3 mm
- net Heartbeat_LED_FP: track 28.8 -> 29.6 mm
- net Fogger_Basin_Float_Switch_FP: track 36.3 -> 37.1 mm
- net Net-(LED9-A): track 2.48 -> 1.88 mm
- added copper zone on In2.Cu, net 12V_FP
- added copper zone on In2.Cu, net 3.3V_FP
- added copper zone on In1.Cu, net GND_FP
Other:
- board text added: "12V IN"
- board text removed: "1K"
- board text removed: "3.3V"
- board text removed: "33"
- board text removed: "Conn_01x0"
- board text removed: "Heartbeat"
- board text removed: "J39"
- board text removed: "TS-1088-AR02016"

Commit message: updated power architecture
Parts:
- moved LED13 32.8 mm to (131.8, 48.0)
- moved R21 32.8 mm to (131.6, 52.7)
- moved C6 12.0 mm to (99.6, 62.7), turned to 180 degrees
- moved C1 10.4 mm to (116.1, 84.9), turned to -90 degrees
- moved D2 9.99 mm to (110.3, 78.4), turned to -90 degrees
- moved C5 9.57 mm to (98.6, 64.7), turned to 180 degrees
- moved L2 9.13 mm to (101.9, 77.1), turned to 180 degrees
- moved C11 9.11 mm to (100.6, 83.6)
- moved C3 9.11 mm to (95.4, 83.6)
- moved C9 9.11 mm to (98.0, 83.6)
- moved R1 8.42 mm to (104.9, 85.2), turned to 0 degrees
- moved C2 7.86 mm to (107.6, 79.0)
- moved C8 7.72 mm to (105.0, 83.5), turned to 180 degrees
- moved R4 5.41 mm to (103.5, 88.1), turned to 0 degrees
- moved R3 5.14 mm to (109.2, 90.6)
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Routing:
- net 12V: track 0.00 -> 38.5 mm, vias 0 -> 37
- net GlycolSol: track 51.9 -> 18.5 mm
- net WaterSol: track 68.2 -> 34.8 mm
- net Circ_Fan: track 47.4 -> 15.6 mm
- net GND_FP: track 8.60 -> 39.4 mm, vias 8 -> 35
- net DrainSol: track 37.9 -> 7.75 mm
- net FoggerSol: track 70.5 -> 42.1 mm
- net Heater Fans: track 61.1 -> 32.9 mm
- net 3.3V: track 3.88 -> 16.8 mm, vias 3 -> 9
- net Net-(D2-K): track 11.8 -> 0.00 mm
- net Net-(J41-Pin_1): track 14.5 -> 23.3 mm
- net 3.3V_FP: track 0.38 -> 8.24 mm, vias 0 -> 6
- net Piezo1: track 41.5 -> 48.8 mm
- net Piezo2: track 45.1 -> 52.4 mm
- net VBUS: track 0.28 -> 6.90 mm
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- added copper zone on F.Cu, net 12V
- added copper zone on F.Cu, net 3.3V
- added copper zone on F.Cu, net GND
- added copper zone on F.Cu, net Net-(D2-K)

Commit message: made some connections
Parts:
- moved C15 3.85 mm to (91.5, 107.4), turned to 90 degrees
- moved R25 2.49 mm to (87.8, 112.5)
- moved C13 2.01 mm to (90.0, 112.7)
- moved C20 0.55 mm to (80.7, 95.2)
- moved R26 0.55 mm to (83.1, 93.2)
Routing:
- net WaterSol: track 34.8 -> 71.0 mm
- net GlycolSol: track 18.5 -> 54.4 mm
- net 3.3V: track 16.8 -> 49.6 mm, vias 9 -> 29
- net Circ_Fan: track 15.6 -> 47.4 mm
- net DrainSol: track 7.75 -> 38.7 mm
- net FoggerSol: track 42.1 -> 72.8 mm
- net GND: track 3.00 -> 32.9 mm, vias 21 -> 42
- net Heater Fans: track 32.9 -> 62.5 mm
- net 12V: track 38.5 -> 42.5 mm, vias 37 -> 40
- net EN: track 97.5 -> 95.4 mm
- net Net-(C4-Pad1): track 0.00 -> 1.73 mm
- net CS_Display: track 40.8 -> 41.7 mm
- net Net-(U8-IO3): track 2.49 -> 3.23 mm
- net External_Fan_PWM: track 19.0 -> 19.6 mm
- net BootMode: track 41.4 -> 41.9 mm

Commit message: started box
Parts:
- removed C16, C17: DNP, easyeda2kicad:C1206
- removed R1, R14, R17, R24, R25, R26, R27, R28, R30, R31, R65, R67, R69, R71, R73, R75: 10k, easyeda2kicad:R0603
- removed U7: TC4428EOA, easyeda2kicad:SOIC-8_L4.9-W3.9-P1.27-LS6.0-BL
- added R40: 10K, easyeda2kicad:R0805, F.Cu at (83.3, 71.2)
- added R41: 10K, easyeda2kicad:R0805, F.Cu at (83.3, 58.4)
- added R42: 10K, easyeda2kicad:R0805, F.Cu at (74.6, 67.2)
- added R44: 10K, easyeda2kicad:R0805, F.Cu at (74.8, 79.8)
- added R48: 10K, easyeda2kicad:R0805, F.Cu at (83.3, 84.4)
- added R49: 10K, easyeda2kicad:R0805, F.Cu at (74.5, 54.3)
- added R50: 10K, easyeda2kicad:R0805, F.Cu at (82.9, 45.9)
- added R51: 10K, easyeda2kicad:R0805, F.Cu at (93.1, 56.1)
- added R52: 10K, easyeda2kicad:R0805, F.Cu at (104.5, 85.1)
- added R53: 10K, easyeda2kicad:R0805, F.Cu at (114.7, 131.6)
- added R54: 10K, easyeda2kicad:R0805, F.Cu at (87.7, 112.7)
- added R55: 10K, easyeda2kicad:R0805, F.Cu at (107.0, 110.8)
- added R56: 10K, easyeda2kicad:R0805, F.Cu at (102.7, 110.2)
- added R57: 10K, easyeda2kicad:R0805, F.Cu at (86.1, 106.5)
- added R59: 10K, easyeda2kicad:R0805, F.Cu at (114.6, 120.0)
- added U1: TC4428EOA713-TUDI, easyeda2kicad:SOIC-8_L4.9-W3.9-P1.27-LS6.0-BL, F.Cu at (96.0, 68.5)
- R61, R63: value 10k -> 10K; footprint easyeda2kicad:R0603 -> easyeda2kicad:R0805
- moved R63 79.0 mm to (156.6, 88.1), turned to 180 degrees
- moved R61 60.0 mm to (114.5, 122.5), turned to 0 degrees
- moved R8 1.54 mm to (90.4, 130.5)
- moved R6 1.49 mm to (90.4, 128.9)
- moved R19 0.76 mm to (118.2, 122.1)
- moved R32 0.62 mm to (165.4, 115.4)
- moved C8 0.43 mm to (105.0, 83.1)
- moved U16 0.42 mm to (80.9, 118.2), turned to 180 degrees
- moved D1 0.35 mm to (146.6, 132.0)
- moved R46 0.22 mm to (89.0, 127.4)
Connections:
- R61 pad 1: GND -> DrainLevel_IO
- R61 pad 2: Net-(J34-Pin_1) -> Drain_Level
- R63 pad 1: GND -> Net-(R63-Pad1)
- R63 pad 2: Net-(J36-Pin_1) -> 3.3V_FP
- SW4 pad 1: Net-(R31-Pad2) -> Net-(R63-Pad1)
- U16 pad 4: D- -> D+
- U16 pad 6: D+ -> D-
- U8 pad 3: Net-(U8-IO2) -> Memory_IO3
- U8 pad 7: Net-(U8-IO3) -> Memory_IO3
Routing:
- net MISO: track 39.8 -> 217.2 mm
- net GND: track 32.9 -> 72.1 mm, vias 42 -> 92
- net 12V_FP: track 71.7 -> 91.0 mm, vias 1 -> 16
- net Memory_IO3: track 0.00 -> 10.6 mm, vias 0 -> 2
- net 3.3V: track 49.6 -> 60.1 mm, vias 29 -> 30
- net GND_FP: track 39.4 -> 48.1 mm, vias 35 -> 38
- net D+: track 26.3 -> 21.8 mm
- net Net-(R63-Pad1): track 0.00 -> 4.38 mm
- net Net-(R31-Pad2): track 4.38 -> 0.00 mm
- net KSD_Fault: track 100.0 -> 96.5 mm
- net D-: track 26.0 -> 22.5 mm
- net Net-(U8-IO3): track 3.23 -> 0.00 mm
- net Net-(U8-IO2): track 2.45 -> 0.00 mm
- net IO19: track 3.94 -> 1.92 mm
- net IO20: track 3.73 -> 2.06 mm
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Other:
- rule pad_to_mask_clearance: 0.1 -> 0
