File: GrowChamberPCB/SwitchingBank.kicad_sch (KiCad schematic)
At the start: 5 parts, among them Q8 BRT30N70P3, Q9 NPN, U11 1N4007W

Commit message: failing to route the board
Parts:
- removed R34: 1k, easyeda2kicad:R0603, symbol easyeda2kicad:FRC0603J102TS
- removed U11: 1N4007W, easyeda2kicad:SOD-123FL_L2.7-W1.8-LS3.7-RD, symbol easyeda2kicad:1N4007W_C7528871
- added J11, J17, J18, J19, J20, J21: TP, TestPoint:TestPoint_Pad_D2.0mm, symbol Connector_Generic:Conn_01x01
- added Q17: NPN, easyeda2kicad:SOT-23-3_L3.0-W1.7-P0.95-LS2.9-BR, symbol easyeda2kicad:2N22221P-TD
- added Q18: MOSFET, easyeda2kicad:SOT-23-3_L2.9-W1.3-P1.90-LS2.4-BR, symbol easyeda2kicad:AO3400A_C347475
- added R34, R53: 1M, easyeda2kicad:R0603, symbol easyeda2kicad:FRC0603F1004TS
- added R52: 1k, easyeda2kicad:R0603, symbol easyeda2kicad:FRC0603J102TS
Connections:
- net 12V: now also R34.1, R53.1
- net GND: now also Q17.2 (E), Q18.2 (S)
- net Heater_ON: now also J17.1 (Pin_1), Q18.3 (D)
- net Heater_Switch: now also J18.1 (Pin_1), R52.1
- net LEDs: now also J20.1 (Pin_1)
- net at Q8.1 (G), Q9.3 (C): now also J19.1 (Pin_1), R34.2
- net GPIO18 renamed LEDIO
- net LEDIO: now also J21.1 (Pin_1)
- new net: J11.1 (Pin_1), Q17.3 (C), Q18.1 (G), R53.2
- new net: Q17.1 (B), R52.2
Other:
- removed sheet MOSFETSwitch6

Commit message: redesign 3
Parts:
- R34, R53: value 1M -> 100k; Manufacturer FOJAN(富捷) -> UNI-ROYAL(Uniroyal Elec)

Commit message: finished routing
Parts:
- removed J11, J17, J18, J19, J20, J21: TP, TestPoint:TestPoint_Pad_D2.0mm, symbol Connector_Generic:Conn_01x01
- removed Q17, Q9: NPN, easyeda2kicad:SOT-23-3_L3.0-W1.7-P0.95-LS2.9-BR, symbol easyeda2kicad:2N22221P-TD
- removed Q18: MOSFET, easyeda2kicad:SOT-23-3_L2.9-W1.3-P1.90-LS2.4-BR, symbol easyeda2kicad:AO3400A_C347475
- removed Q8: BRT30N70P3, easyeda2kicad:TO-252-2_L6.6-W6.1-P4.60-LS10.0-BR-CW, symbol easyeda2kicad:BRT30N70P3
- removed R32, R52: 1k, easyeda2kicad:R0603, symbol easyeda2kicad:FRC0603J102TS
- removed R34, R53: 100k, easyeda2kicad:R0603, symbol easyeda2kicad:FRC0603F1004TS
Other:
- removed sheet MOSFETSwitch
- removed sheet MOSFETSwitch1
- removed sheet MOSFETSwitch2
- removed sheet MOSFETSwitch3
- removed sheet MOSFETSwitch4
- removed sheet MOSFETSwitch5
- added sheet Untitled Sheet (MOSFETSwitch.kicad_sch)
- added sheet Untitled Sheet1 (MOSFETSwitch.kicad_sch)
- added sheet Untitled Sheet2 (MOSFETSwitch.kicad_sch)
- added sheet Untitled Sheet3 (MOSFETSwitch.kicad_sch)
- added sheet Untitled Sheet4 (MOSFETSwitch.kicad_sch)
- added sheet Untitled Sheet5 (MOSFETSwitch.kicad_sch)
- added sheet Untitled Sheet6 (MOSFETSwitch.kicad_sch)
- added sheet Untitled Sheet7 (MOSFETSwitch.kicad_sch)
- note removed: "LED Driver"
