File: GrowChamberPCB/3.3VESD.kicad_sch (KiCad schematic)
At the start: 1 part

Commit message: finished routing
Parts:
- removed D13: SRV05-4_C2836319, easyeda2kicad:SOT-23-6_L2.9-W1.6-P0.95-LS2.8-BL, symbol easyeda2kicad:SRV05-4_C2836319
- added U11: SRV05-4A, easyeda2kicad:SOT-23-6_L2.9-W1.6-P0.95-LS2.9-BL, symbol easyeda2kicad:SRV05-4A_C20615829
Connections:
- net 3.3V_FP: now also U11.5 (VP)
- net GND_FP: now also U11.2 (VN)
- net IO1: now also U11.1 (I/O)
- net IO2: now also U11.3 (I/O)
- net IO3: now also U11.6 (I/O)
- net IO4: now also U11.4 (I/O)
Changed lines of the file:
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@@
 	(global_label "3.3V_FP"
 		(shape input)
-		(at 128.27 102.87 180)
+		(at 130.81 102.87 180)
 		(fields_autoplaced yes)
 		(effects
@@
 		)
 		(property "Intersheetrefs" "${INTERSHEET_REFS}"
-			(at 117.8462 102.87 0)
+			(at 120.3862 102.87 0)
 			(hide yes)
 			(show_name no)
@@
 		)
 	)
+	(global_label "Display_Reset"
+		(shape input)
+		(at 15.5271 1.3498 180)
+		(fields_autoplaced yes)
+		(effects
+			(font
+				(size 1.27 1.27)
+			)
+			(justify right)
+		)
+		(property "Intersheetrefs" "${INTERSHEET_REFS}"
+			(at -0.4604 1.3498 0)
+			(hide yes)
+			(show_name no)
+			(do_not_autoplace no)
+			(effects
+				(font
+					(size 1.27 1.27)
+				)
+				(justify right)
+			)
+		)
+	)
 	(global_label "GND_FP"
 		(shape input)
-		(at 161.29 102.87 0)
+		(at 156.21 102.87 0)
 		(fields_autoplaced yes)
 		(effects
@@
 		)
 		(property "Intersheetrefs" "${INTERSHEET_REFS}"
-			(at 171.4719 102.87 0)
+			(at 166.3919 102.87 0)
 			(hide yes)
 			(show_name no)
@@
 	(hierarchical_label "IO2"
 		(shape input)
-		(at 161.29 92.71 0)
+		(at 156.21 97.79 0)
 		(effects
 			(font
@@
 	(hierarchical_label "IO1"
 		(shape input)
-		(at 161.29 113.03 0)
+		(at 156.21 107.95 0)
 		(effects
 			(font
@@
 	(hierarchical_label "IO4"
 		(shape input)
-		(at 128.27 92.71 180)
+		(at 130.81 97.79 180)
 		(effects
 			(font
@@
 	(hierarchical_label "IO3"
 		(shape input)
-		(at 128.27 113.03 180)
+		(at 130.81 107.95 180)
 		(effects
 			(font
@@
 	)
 	(symbol
-		(lib_id "easyeda2kicad:SRV05-4_C2836319")
-		(at 144.78 102.87 0)
+		(lib_id "easyeda2kicad:SRV05-4A_C20615829")
+		(at 143.51 102.87 90)
 		(unit 1)
 		(body_style 1)
@@
 		(dnp no)
 		(fields_autoplaced yes)
-		(property "Reference" "D13"
-			(at 144.78 78.74 0)
-			(show_name no)
-			(do_not_autoplace no)
-			(effects
-				(font
-					(size 1.27 1.27)
-				)
-			)
-		)
-		(property "Value" "SRV05-4_C2836319"
-			(at 144.78 81.28 0)
-			(show_name no)
-			(do_not_autoplace no)
-			(effects
-				(font
-					(size 1.27 1.27)
-				)
-			)
-		)
-		(property "Footprint" "easyeda2kicad:SOT-23-6_L2.9-W1.6-P0.95-LS2.8-BL"
-			(at 144.78 120.65 0)
-			(hide yes)
-			(show_name no)
-			(do_not_autoplace no)
-			(effects
-				(font
-					(size 1.27 1.27)
-				)
-			)
-		)
-		(property "Datasheet" "https://www.lcsc.com/datasheet/C2836319.pdf"
-			(at 144.78 123.19 0)
+		(property "Reference" "U11"
+			(at 143.51 87.63 90)
+			(show_name no)
+			(do_not_autoplace no)
+			(effects
+				(font
+					(size 1.27 1.27)
+				)
+			)
+		)
+		(property "Value" "SRV05-4A"
+			(at 143.51 90.17 90)
+			(show_name no)
+			(do_not_autoplace no)
+			(effects
+				(font
+					(size 1.27 1.27)
+				)
+			)
+		)
+		(property "Footprint" "easyeda2kicad:SOT-23-6_L2.9-W1.6-P0.95-LS2.9-BL"
+			(at 163.83 102.87 0)
+			(hide yes)
+			(show_name no)
+			(do_not_autoplace no)
+			(effects
+				(font
+					(size 1.27 1.27)
+				)
+			)
+		)
+		(property "Datasheet" "https://www.lcsc.com/datasheet/C20615829.pdf"
+			(at 166.37 102.87 0)
 			(hide yes)
 			(show_name no)
@@
 		)
 		(property "Description" ""
-			(at 144.78 102.87 0)
-			(hide yes)
-			(show_name no)
-			(do_not_autoplace no)
-			(effects
-				(font
-					(size 1.27 1.27)
-				)
-			)
-		)
-		(property "Manufacturer" "MSKSEMI(美森科)"
-			(at 144.78 125.73 0)
-			(hide yes)
-			(show_name no)
-			(do_not_autoplace no)
-			(effects
-				(font
-					(size 1.27 1.27)
-				)
-			)
-		)
-		(property "MPN" "SRV05-4"
-			(at 144.78 128.27 0)
-			(hide yes)
-			(show_name no)
-			(do_not_autoplace no)
-			(effects
-				(font
-					(size 1.27 1.27)
-				)
-			)
-		)
-		(property "LCSC Part" "C2836319"
-			(at 144.78 130.81 0)
-			(hide yes)
-			(show_name no)
-			(do_not_autoplace no)
-			(effects
-				(font
-					(size 1.27 1.27)
-				)
-			)
-		)
-		(property "Basic Part?" ""
-			(at 144.78 102.87 0)
-			(hide yes)
-			(show_name no)
-			(do_not_autoplace no)
-			(effects
-				(font
-					(size 1.27 1.27)
-				)
-			)
-		)
-		(property "MFG Part Number" ""
-			(at 144.78 102.87 0)
-			(hide yes)
-			(show_name no)
-			(do_not_autoplace no)
-			(effects
-				(font
-					(size 1.27 1.27)
-				)
-			)
-		)
-		(property "Package" ""
-			(at 144.78 102.87 0)
-			(hide yes)
-			(show_name no)
-			(do_not_autoplace no)
-			(effects
-				(font
-					(size 1.27 1.27)
-				)
-			)
-		)
-		(property "Type (SMD/thru-hole, etc.)" ""
-			(at 144.78 102.87 0)
+			(at 143.51 102.87 0)
+			(hide yes)
+			(show_name no)
+			(do_not_autoplace no)
+			(effects
+				(font
+					(size 1.27 1.27)
+				)
+			)
+		)
+		(property "Manufacturer" "R+O(宏嘉诚)"
+			(at 168.91 102.87 0)
+			(hide yes)
+			(show_name no)
+			(do_not_autoplace no)
+			(effects
+				(font
+					(size 1.27 1.27)
+				)
+			)
+		)
+		(property "MPN" "SRV05-4A"
+			(at 171.45 102.87 0)
+			(hide yes)
+			(show_name no)
+			(do_not_autoplace no)
+			(effects
+				(font
+					(size 1.27 1.27)
+				)
+			)
+		)
+		(property "LCSC Part" "C20615829"
+			(at 173.99 102.87 0)
 			(hide yes)
 			(show_name no)
@@
 		(pin "1"
 		)
+		(pin "6"
+		)
+		(pin "5"
+		)
+		(pin "3"
+		)
+		(pin "4"
+		)
 		(pin "2"
-		)
-		(pin "3"
-		)
-		(pin "6"
-		)
-		(pin "5"
-		)
-		(pin "4"
 		)
 		(instances
 			(project "GrowChamberPCB"
+				(path "/e884bae1-e2d9-44d2-8169-161aa31a84ae/23dbc102-7df9-49e8-b89b-2ac86618ae12/022f2755-8e55-497d-96c2-53ffea4d6ddf"
+					(reference "U17")
+					(unit 1)
+				)
+				(path "/e884bae1-e2d9-44d2-8169-161aa31a84ae/23dbc102-7df9-49e8-b89b-2ac86618ae12/ce919896-a754-4b15-8f81-0077b8c32c9e"
+					(reference "U14")
+					(unit 1)
+				)
+				(path "/e884bae1-e2d9-44d2-8169-161aa31a84ae/23dbc102-7df9-49e8-b89b-2ac86618ae12/e352a733-7762-4798-9493-913f0607de0b"
+					(reference "U16")
+					(unit 1)
+				)
+				(path "/e884bae1-e2d9-44d2-8169-161aa31a84ae/23dbc102-7df9-49e8-b89b-2ac86618ae12/faebad59-de3b-4399-b041-528b99636dd1"
+					(reference "U18")
+					(unit 1)
+				)
 				(path "/e884bae1-e2d9-44d2-8169-161aa31a84ae/c2403359-39ea-416b-9a92-81a595d10d09/4617caea-6164-4cde-afba-3767557ebe60"
-					(reference "D16")
+					(reference "U12")
 					(unit 1)
 				)
 				(path "/e884bae1-e2d9-44d2-8169-161aa31a84ae/c2403359-39ea-416b-9a92-81a595d10d09/523196bc-63c3-40bf-aa15-5a19eeb2813e"
-					(reference "D13")
+					(reference "U11")
+					(unit 1)
+				)
+				(path "/e884bae1-e2d9-44d2-8169-161aa31a84ae/c2403359-39ea-416b-9a92-81a595d10d09/e3523d29-de98-4a92-b088-8f1fc0f3a344"
+					(reference "U15")
 					(unit 1)
 				)
 				(path "/e884bae1-e2d9-44d2-8169-161aa31a84ae/c2403359-39ea-416b-9a92-81a595d10d09/f371a2c8-8593-49e6-b7f8-2b57ddd687f3"
-					(reference "D17")
-					(unit 1)
-				)
+					(reference "U13")
+					(unit 1)
+				)

Commit message: fixing stuff
Connections:
- net 3.3V_FP renamed GND
- net GND_FP renamed Power
Changed lines of the file:
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@@
 	(generator_version "10.0")
 	(paper "A4")
-	(global_label "3.3V_FP"
-		(shape input)
-		(at 130.81 102.87 180)
-		(fields_autoplaced yes)
-		(effects
-			(font
-				(size 1.27 1.27)
-			)
-			(justify right)
-		)
-		(property "Intersheetrefs" "${INTERSHEET_REFS}"
-			(at 120.3862 102.87 0)
-			(hide yes)
-			(show_name no)
-			(do_not_autoplace no)
-			(effects
-				(font
-					(size 1.27 1.27)
-				)
-				(justify right)
-			)
-		)
-	)
 	(global_label "Display_Reset"
 		(shape input)
@@
 		)
 	)
-	(global_label "GND_FP"
-		(shape input)
-		(at 156.21 102.87 0)
-		(fields_autoplaced yes)
-		(effects
-			(font
-				(size 1.27 1.27)
-			)
-			(justify left)
-		)
-		(property "Intersheetrefs" "${INTERSHEET_REFS}"
-			(at 166.3919 102.87 0)
-			(hide yes)
-			(show_name no)
-			(do_not_autoplace no)
-			(effects
-				(font
-					(size 1.27 1.27)
-				)
-				(justify left)
-			)
-		)
-	)
 	(hierarchical_label "IO2"
 		(shape input)
@@
 			)
 			(justify left)
+		)
+	)
+	(hierarchical_label "GND"
+		(shape input)
+		(at 130.81 102.87 180)
+		(effects
+			(font
+				(size 1.27 1.27)
+			)
+			(justify right)
 		)
 	)
@@
 		)
 	)
+	(hierarchical_label "Power"
+		(shape input)
+		(at 156.21 102.87 0)
+		(effects
+			(font
+				(size 1.27 1.27)
+			)
+			(justify left)
+		)
+	)
